File: KiCAD/286.kicad_sch (KiCad schematic)
At the start: 37 parts, among them CON1 Conn_02x20_Odd_Even, CON2 Conn_02x17_Odd_Even, U1 74LS00, U14 7406, U15 HM6818P, U16 4069, U19 D8041AHC, U2 74LS00, U7 N80L286-16/S, X1 Crystal, X2 Crystal

Commit message: DPS update
Parts:
- removed U14: 7406, Package_DIP:DIP-14_W7.62mm, symbol 74xx_IEEE:7406
- removed U2: 74LS00, symbol 74xx:74LS00
- added C41, C43, C44, C45: ~, Capacitor_THT:C_Disc_D4.3mm_W1.9mm_P5.00mm, symbol Device:C_Small
- added D1: D_Small, Diode_THT:D_A-405_P10.16mm_Horizontal, symbol Device:D_Small
- added JP1, JP7: Conn_01x03, Connector_PinHeader_2.54mm:PinHeader_1x03_P2.54mm_Vertical, symbol Connector_Generic:Conn_01x03
- added JP10, JP14, JP15, JP2, JP5: Conn_01x02, Connector_PinSocket_2.54mm:PinSocket_1x02_P2.54mm_Vertical, symbol Connector_Generic:Conn_01x02
- added RP1: R_Network09, Resistor_THT:R_Array_SIP10, symbol Device:R_Network09
- added U1, U18, U3: 74LS245, Package_DIP:DIP-20_W7.62mm, symbol 74xx:74LS245
- added U14: 74LS06, Package_DIP:DIP-14_W7.62mm, symbol 74xx:74LS06
- added U20: PAL16L8, Package_DIP:DIP-20_W7.62mm, symbol Logic_Programmable:PAL16L8
- added U8: ~, Package_LCC:PLCC-68, symbol _mine_d:MCS2301
- renumbered U1 to U100
Connections:
- net A11: now also U7.18 (A13)
- net GND: now also U1.10 (GND), U14.7 (GND), U18.10 (GND), U20.10 (GND), U3.10 (GND)
- net VCC: now also U14.14 (VCC)
- net VDD: now also U1.20 (VCC), U18.20 (VCC), U20.20 (VCC), U3.20 (VCC)
- net u1-1: now also U1.1 (A->B)
- net u1-3: now also U1.3 (A1)
- net u14-13: now also U14.13
- net u14-5: now also U14.5
- net u14-6: now also U14.6
- net u16-12: now also U14.11
- net con1-10: now reaches CON1.10 (Pin_10)
- net con1-10: now also U3.6 (A4)
- net u1-5: now reaches CON1.11 (Pin_11)
- net u1-5: now also U1.5 (A3)
- net con1-12: now reaches CON1.12 (Pin_12)
- net con1-12: now also U3.5 (A3)
- net con1-14: now reaches CON1.14 (Pin_14)
- net con1-14: now also U3.4 (A2)
- net con1-16: now reaches CON1.16 (Pin_16)
- net con1-16: now also U3.3 (A1)
- net con1-18: now reaches CON1.18 (Pin_18)
- net con1-18: now also U3.2 (A0)
- net con1-23: now reaches CON1.23 (Pin_23)
- net con1-25: now reaches CON1.25 (Pin_25)
- net con1-31: now reaches CON1.31 (Pin_31)
- net con1-33: now reaches CON1.33 (Pin_33)
- net con1-35: now reaches CON1.35 (Pin_35)
- net con1-37: now reaches CON1.37 (Pin_37)
- net con1-4: now reaches CON1.4 (Pin_4)
- net con1-4: now also U3.9 (A7)
- net con1-5: now reaches CON1.5 (Pin_5)
- net con1-6: now reaches CON1.6 (Pin_6)
- net con1-6: now also U3.8 (A6)
- net con1-7: now reaches CON1.7 (Pin_7)
- net con1-8: now reaches CON1.8 (Pin_8)
- net con1-8: now also U3.7 (A5)
- net u1-6: now reaches CON1.9 (Pin_9)
- net u1-6: now also U1.6 (A4)
- net u8-61: now reaches CON2.20 (Pin_20)
- net u8-61: now also U8.61 (~{STEP})
- net u8-59: now reaches CON2.22 (Pin_22)
- net u8-59: now also U8.59 (~{WD})
- net u8-63: now reaches CON2.26 (Pin_26)
- net u8-63: now also RP1.4 (R3), U8.63 (~{TRAK0})
- net u8-64: now reaches CON2.28 (Pin_28)
- net u8-64: now also RP1.9 (R8), U8.64 (~{WP})
- net u8-65: now reaches CON2.30 (Pin_30)
- net u8-65: now also RP1.8 (R7), U8.65 (~{RDATA})
- net con2-34: now reaches CON2.34 (Pin_34)
- net u8-62: now reaches CON2.8 (Pin_8)
- net u8-62: now also RP1.7 (R6), U8.62 (~{INDEX})
- new net d1-2: D1.2 (A)
- new net jp1-1: JP1.1 (Pin_1)
- new net jp1-2: JP1.2 (Pin_2)
- new net jp1-3: JP1.3 (Pin_3)
- new net jp15-1: JP15.1 (Pin_1)
- new net jp2-1: JP2.1 (Pin_1), JP7.2 (Pin_2)
- new net rp1-10: RP1.10 (R9)
- new net rp1-6: RP1.6 (R5)
- new net u1-19: U1.19 (CE)
- new net u1-2: U1.2 (A0)
- new net u18-1: U18.1 (A->B)
- new net u18-11: U18.11 (B7)
- new net u18-12: U18.12 (B6)
- new net u18-13: U18.13 (B5)
- new net u18-14: U18.14 (B4)
- new net u18-15: U18.15 (B3)
- new net u18-16: U18.16 (B2)
- new net u18-17: U18.17 (B1)
- new net u18-18: U18.18 (B0)
- new net u18-2: U18.2 (A0)
- new net u18-3: U18.3 (A1)
- new net u18-4: U18.4 (A2)
- new net u18-5: U18.5 (A3)
- new net u18-6: U18.6 (A4)
- new net u18-8: U18.8 (A6)
- new net u20-11: U20.11 (I10)
- new net u20-14: U20.14 (IO6)
- new net u20-15: U20.15 (IO5)
- new net u20-17: U20.17 (I03)
- new net u20-18: U20.18 (IO2)
- new net u20-19: U20.19 (IO1)
- new net u20-2: U20.2 (I2)
- new net u20-3: U20.3 (I3)
- new net u20-5: U20.5 (I5)
- new net u20-8: U20.8 (I8), U8.9 (SA8)
- new net u20-9: U20.9 (I9)
- new net u3-11: U3.1 (A->B), U3.11 (B7)
- new net u3-12: U3.12 (B6)
- new net u3-16: U3.16 (B2)
- new net u3-18: U3.18 (B0)
- new net u3-19: U3.19 (CE)
- new net u8-48: U8.48 (~{MO1})
- new net u8-49: U8.49 (~{MO0})
- new net u8-51: U8.51 (~{DS1})
- new net u8-55: U8.55 (~{DIR})
- new net u8-66: RP1.5 (R4), U8.66 (~{DSKCHNG})
Other:
- moved on the sheet: CON1, CON2, JP19, U100B, U100C, U100D, U100E

Commit message: PCB update
Parts:
- added BKSW1: B, Connector_PinHeader_2.54mm:PinHeader_1x03_P2.54mm_Vertical, symbol Connector_Generic:Conn_01x03
- added BKSW2: K, Connector_PinHeader_2.54mm:PinHeader_1x03_P2.54mm_Vertical, symbol Connector_Generic:Conn_01x03
- added BKSW3: J, Connector_PinHeader_2.54mm:PinHeader_1x03_P2.54mm_Vertical, symbol Connector_Generic:Conn_01x03
- added BKSW4: P, Connector_PinHeader_2.54mm:PinHeader_1x03_P2.54mm_Vertical, symbol Connector_Generic:Conn_01x03
- added C32, C50: ~, Capacitor_THT:C_Disc_D4.3mm_W1.9mm_P5.00mm, symbol Device:C_Small
- added C37: 10u, Capacitor_THT:CP_Radial_D5.0mm_P2.50mm, symbol Device:C_Polarized_Small
- added R2: R_Small, Resistor_THT:R_Axial_DIN0204_L3.6mm_D1.6mm_P5.08mm_Horizontal, symbol Device:R_Small
- added RP10, RP11: R_Network04, Resistor_THT:R_Array_SIP5, symbol Device:R_Network04
- added RP8: R_Network07, Resistor_THT:R_Array_SIP8, symbol Device:R_Network07
Connections:
- net osc2-out: now also U8.33 (XTAL1)
- net u1-1: now also U3.1 (A->B); no longer U100.1, U100.2
- net u1-3: no longer U100.3
- net u3-11: no longer U3.1 (A->B)
- net u8-1: now reaches U8.1 (SA0)
- net u8-10: now reaches U8.10 (SA9)
- net u8-11: now reaches U8.11 (AEN)
- net u8-2: now reaches U8.2 (SA1)
- net u8-23: now reaches U8.23 (DRQ)
- net u8-24: now reaches U8.24 (~{IOW})
- net u8-25: now reaches U8.25 (~{IOR})
- net u8-26: now reaches U8.26 (IRQ)
- net u8-27: now reaches U8.27 (~{DACK})
- net u8-28: now reaches U8.28 (T/C)
- net u8-3: now reaches U8.3 (SA2)
- net u8-4: now reaches U8.4 (SA3)
- net u8-5: now reaches U8.5 (SA4)
- net u8-53: now reaches U8.53 (~{WE})
- net u8-58: now reaches U8.58 (~{RWC})
- net u8-6: now reaches U8.6 (SA5)
- net u8-7: now reaches U8.7 (SA6)
- net u8-8: now reaches U8.8 (SA7)
- net rp1-2: now reaches RP1.2 (R1)
- net u1-12 renamed u100-12
- net u1-4 renamed u100-4
- net u1-8 renamed u100-8
- net u1-9 renamed u100-9
- new net bk1-1: BKSW1.1 (Pin_1)
- new net bk1-3: BKSW1.3 (Pin_3)
- new net bk2-1: BKSW2.1 (Pin_1)
- new net bk2-2: BKSW2.2 (Pin_2)
- new net bk2-3: BKSW2.3 (Pin_3)
- new net bk3-1: BKSW3.1 (Pin_1)
- new net bk3-3: BKSW3.3 (Pin_3)
- new net bk4-1: BKSW4.1 (Pin_1)
- new net bk4-2: BKSW4.2 (Pin_2)
- new net bk4-3: BKSW4.3 (Pin_3)
- new net pr11-3: RP11.3 (R2)
- new net rp10-2: RP10.2 (R1)
- new net rp10-3: RP10.3 (R2)
- new net rp10-4: RP10.4 (R3)
- new net rp8-2: RP8.2 (R1)
- new net rp8-4: RP8.4 (R3)
- new net rp8-6: RP10.5 (R4), RP8.6 (R5)
- new net u100-1: U100.1, U100.2
- new net u100-3: U100.3
Other:
- moved on the sheet: D1, JP1, JP10, JP14, JP15, JP19, JP2, JP20, JP5, JP7, KEYBOARD1, R18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

Commit message: PCB update
Parts:
- added D2: D_Small, Diode_THT:D_A-405_P10.16mm_Horizontal, symbol Device:D_Small
- added J12: Bus_ISA_16bit, _mine:ISA_16bit, symbol Connector:Bus_ISA_16bit
- added JP11: Conn_01x02, Connector_PinSocket_2.54mm:PinSocket_1x02_P2.54mm_Vertical, symbol Connector_Generic:Conn_01x02
- added R14, R17, R53: R_Small, Resistor_THT:R_Axial_DIN0204_L3.6mm_D1.6mm_P5.08mm_Horizontal, symbol Device:R_Small
- added RA2: R_Network08, Resistor_THT:R_Array_SIP9, symbol Device:R_Network08
Connections:
- net VCC is gone; now on net VDD: U100.14 (VCC), U14.14 (VCC), U15.20 (CKFS), U15.24 (VDD), U16.14 (VDD)
- net VDD: now also D2.1 (K)
- net u3-18: now also J12.98 (D15)
- net con1-25 renamed j12-ior
- net j12-ior: now also J12.14 (~{IOR})
- net rp10-4 renamed j12-memr
- net j12-memr: now also J12.89 (~{MEMR})
- net u20-11 renamed j12-aen
- net j12-aen: now also J12.42 (AEN)
- new net +12V: J12.9 (+12V)
- new net -12V: J12.7 (-12V)
- new net -5V: J12.5 (-5V)
- new net j12-ba10: J12.52 (BA10)
- new net j12-ba11: J12.51 (BA11)
- new net j12-ba12: J12.50 (BA12)
- new net j12-ba13: J12.49 (BA13)
- new net j12-ba14: J12.48 (BA14)
- new net j12-ba4: J12.58 (BA04)
- new net j12-ba6: J12.56 (BA06)
- new net j12-ba7: J12.55 (BA07)
- new net j12-dack0: J12.70 (~{DACK0})
- new net j12-drq1: J12.18 (DRQ1)
- new net j12-io: J12.32 (IO)
- new net j12-iocs16: J12.64 (~{IOCS16})
- new net j12-irq4: J12.24 (IRQ4)
- new net j12-master: J12.79 (MASTER)
- new net j12-memcs16: J12.63 (~{MEMCS16})
- new net jp11-1: JP11.1 (Pin_1)
- new net r14-2: R14.2
- new net r17-1: R17.1
- new net ra2-2: RA2.2 (R1)
- new net ra2-3: RA2.3 (R2)
- new net ra2-4: RA2.4 (R3)
- new net ra2-6: RA2.6 (R5)
- new net ra2-7: RA2.7 (R6)
- new net ra2-8: RA2.8 (R7)
- new net ra2-9: RA2.9 (R8)

Commit message: PCB update
Parts:
- added C17, C18, C25: ~, Capacitor_THT:C_Disc_D4.3mm_W1.9mm_P5.00mm, symbol Device:C_Small
- added C19: 10u, Capacitor_THT:CP_Radial_D5.0mm_P2.50mm, symbol Device:C_Polarized_Small
- added Q4: 2SC1815, Package_TO_SOT_THT:TO-92_Inline_Wide, symbol Transistor_BJT:2SC1815
- added R1, R61, R62: R_Small, Resistor_THT:R_Axial_DIN0204_L3.6mm_D1.6mm_P5.08mm_Horizontal, symbol Device:R_Small
- U5: value ~ -> 80C287
- U8: value ~ -> MCS3201FN
Connections:
- net r17-1 is gone; now on net ~{IO}: R17.1
- net u100-8 is gone; now on net ~{BUSY}: U100.8
- net u5-16 is gone; now on net D7: U5.16
- net u5-17 is gone; now on net D6: U5.17
- net u5-18 is gone; now on net D5: U5.18
- net u5-19 is gone; now on net D4: U5.19
- net u5-21 is gone; now on net D2: U5.21
- net u5-22 is gone; now on net D1: U5.22
- net u5-23 is gone; now on net D0: U5.23
- net u5-24 is gone; now on net PEREQ: U5.24
- net u5-36 is gone; now on net ~{PEACK}: U5.36
- net u5-37 is gone; now on net u7-clk: U5.37
- net u5-38 is gone; now on net HLDA: U5.38
- net u5-40 is gone; now on net ~{READY}: U5.40
- net u5-6 is gone; now on net D14: U5.6
- net A11: no longer U7.18 (A13)
- net CAP: now also C17.2
- net VDD: no longer D2.1 (K), U15.20 (CKFS), U15.24 (VDD), U16.14 (VDD)
- net CLK renamed u7-clk
- new net A13: U7.18 (A13)
- new net VBAT: D2.1 (K), U15.20 (CKFS), U15.24 (VDD), U16.14 (VDD)
- new net r61-2: R61.2
Other:
- moved on the sheet: RA2, RP10, RP11, RP8

Commit message: PCB update
Parts:
- added OSC3: DNP, Oscillator:Oscillator_DIP-14, symbol Oscillator:OCXO-14
- added U6: ST62C241-A, Package_QFP:PQFP-160_28x28mm_P0.65mm, symbol _mine_d:ST62C241-A
- Q4: footprint Package_TO_SOT_THT:TO-92_Inline_Wide -> Package_TO_SOT_THT:TO-92_Inline
Connections:
- net jp11-1 is gone; now on net osc1-out: JP11.1 (Pin_1)
- net ra2-4 is gone; now on net ~{BHE}: RA2.4 (R3)
- net A0: now also U6.18
- net A1: now also U6.17
- net A11: now also U6.157
- net A12: now also U6.156
- net A13: now also U6.155
- net A14: now also U6.154
- net A15: now also U6.153
- net A16: now also U6.152
- net A17: now also U6.151
- net A18: now also U6.150
- net A19: now also U6.149
- net A20: now also U6.147
- net A21: now also U6.146
- net A22: now also U6.145
- net A23: now also U6.144
- net A4: now also U6.8
- net A5: now also U6.7
- net A6: now also U6.6
- net A7: now also U6.5
- net A8: now also U6.4
- net A9: now also U6.3
- net D15: now also U6.75
- net HLDA: now also U6.28
- net HOLD: now also U6.27
- net osc2-out: now also JP11.2 (Pin_2)
- net u15-5: now also U6.70
- net u15-6: now also U6.69
- net u19-15: now also U6.68
- net u19-16: now also U6.67
- net u19-17: now also U6.66
- net u19-18: now also U6.65
- net u19-19: now also U6.64
- net u7-clk: now also JP20.3 (Pin_3), R14.1
- net x1-1: now also R44.1
- net ~{BHE}: now also U6.16
- net ~{IO}: now also U6.15
- net ~{READY}: now also U6.26
- net r1-2: now reaches R1.2
- net osc1-out: now reaches OSC1.8 (OUT)
- net osc1-out: now also U6.158
- net u6-39: now reaches R2.2
- net u6-39: now also U6.39
- net r14-2 renamed u6-25
- net u6-25: now also U6.25
- net ra2-3 renamed u6-13
- net u6-13: now also U6.13
- net ra2-6 renamed u6-145
- net u6-145: now also U6.14
- net ra2-7 renamed u6-37
- net u6-37: now also U6.37
- net ra2-8 renamed u6-36
- net u6-36: now also U6.36
- net ra2-9 renamed u6-24
- net u6-24: now also U6.24
- net rp10-2 renamed u6-34
- net u6-34: now also U6.34
- net rp10-3 renamed u6-35
- net u6-35: now also U6.35
- net u100-12 renamed u6-29
- net u6-29: now also U6.29
- net u18-1 renamed u6-72
- net u6-72: now also U6.72
- new net osc3-out: OSC3.8 (OUT), U6.62
- new net u6-10: U6.10
- new net u6-12: U6.12
- new net u6-148: U6.148
- new net u6-2: U6.2
- new net u6-22: U6.22
- new net u6-30: U6.30
- new net u6-31: U6.31
- new net u6-32: U6.32
- new net u6-33: U6.33
- new net u6-38: U6.38
- new net u6-55: U6.55
- new net u6-71: U6.71
- new net u6-73: U6.73
- new net u6-74: U6.74
- new net u6-76: U6.76
- new net u6-77: U6.77
- new net u6-78: U6.78
- new net u6-81: U6.81
- new net u6-82: U6.82
- new net u6-85: U6.85
- new net u6-87: U6.87
- new net u6-88: U6.88

Commit message: PCB update
Parts:
- removed RP8: R_Network07, Resistor_THT:R_Array_SIP8, symbol Device:R_Network07
- added RP8: R_Pack04_SIP, Resistor_THT:R_Array_SIP8, symbol Device:R_Pack04_SIP
- Q4: footprint Package_TO_SOT_THT:TO-92_Inline -> Package_TO_SOT_THT:TO-92_Inline_Wide
Connections:
- net bk1-1 is gone; now on net u6-127: BKSW1.1 (Pin_1)
- net bk1-3 is gone; now on net u6-126: BKSW1.3 (Pin_3)
- net bk2-1 is gone; now on net u6-119: BKSW2.1 (Pin_1)
- net bk2-3 is gone; now on net u6-118: BKSW2.3 (Pin_3)
- net bk3-1 is gone; now on net u6-125: BKSW3.1 (Pin_1)
- net bk3-3 is gone; now on net u6-124: BKSW3.3 (Pin_3)
- net bk4-3 is gone; now on net u6-116: BKSW4.3 (Pin_3)
- net d1-2 is gone; now on net u6-53: D1.2 (A)
- net jp20-1 is gone; now on net u6-22: JP20.1 (Pin_1)
- net r1-2 is gone; now on net u6-11: R1.2
- net r61-2 is gone; now on net u6-140: R61.2
- net ra2-2 is gone; now on net u6-61: RA2.2 (R1)
- net u19-21 is gone; now on net u6-60: U19.21 (P20)
- net u19-22 is gone; now on net u6-59: U19.22 (P21)
- net u5-1 is gone; now on net ~{S1}: U5.1
- net u5-2 is gone; now on net ~{S0}: U5.2
- net u5-3 is gone; now on net COT~{INTA}: U5.3
- net u6-10 is gone; now on net A2: U6.10
- net u6-12 is gone; now on net RESET: U6.12
- net u6-13 is gone; now on net COT~{INTA}: RA2.3 (R2), U6.13
- net u6-145 is gone; now on net ~{S1}: RA2.6 (R5), U6.14
- net u6-2 is gone; now on net A10: U6.2
- net u6-24 is gone; now on net ~{S0}: RA2.9 (R8), U6.24
- net u6-76 is gone; now on net D7: U6.76
- net u6-81 is gone; now on net VDD: U6.81
- net u6-87 is gone; now on net D13: U6.87
- net u6-88 is gone; now on net D5: U6.88
- net A3: now also U6.9
- net D0: now also U6.111
- net D1: now also U6.107
- net D10: now also U6.102
- net D11: now also U6.95
- net D12: now also U6.91
- net D14: now also U6.83
- net D2: now also U6.103
- net D3: now also U6.96
- net D4: now also U6.92
- net D6: now also U6.84
- net D8: now also U6.110
- net D9: now also U6.106
- net GND: now also C17.1, C27.2, C28.1, C46.1, C47.1, JP19.3 (Pin_3), OSC1.7 (GND), OSC2.7 (GND), OSC3.7 (GND), Q4.1 (E), R18.2, U6.101, U6.121, U6.122, U6.159, U6.160, U6.19, U6.21, U6.41, U6.42, U6.63, U6.79, U6.80, U6.99
- net PEREQ: now also R18.1
- net VDD: now also C28.2, JP19.1 (Pin_1), R17.2, RA2.1 (common), RP10.1 (common), RP11.1 (common), U6.1, U6.100, U6.120, U6.20, U6.40
- net j12-iocs16: now also U6.57
- net j12-memcs16: now also U6.56
- net rp8-2: now also RP8.2 (R1.2)
- net rp8-4: now also RP8.4 (R2.2)
- net rp8-6: now also RP8.6 (R3.2)
- net r1-1: now reaches R1.1
- net r1-1: now also Q4.3 (B)
- net ra2-5: now reaches RA2.5 (R4)
- net q4-2: now reaches Q4.2 (C)
- net u6-104: now reaches U6.104
- net u6-105: now reaches U6.105
- net u6-108: now reaches U6.108
- net u6-109: now reaches U6.109
- net u6-11: now reaches U6.11
- net u6-112: now reaches U6.112
- net u6-113: now reaches U6.113
- net u6-114: now reaches U6.114
- net u6-115: now reaches U6.115
- net u6-116: now reaches U6.116
- net u6-117: now reaches U6.117
- net u6-118: now reaches U6.118
- net u6-119: now reaches U6.119
- net u6-123: now reaches U6.123
- net u6-124: now reaches U6.124
- net u6-124: now also U6.142
- net u6-125: now reaches U6.125
- net u6-126: now reaches U6.126
- net u6-127: now reaches U6.127
- net u6-128: now reaches U6.128
- net u6-129: now reaches U6.129
- net u6-130: now reaches U6.130
- net u6-131: now reaches U6.131
- net u6-132: now reaches U6.132
- net u6-133: now reaches U6.133
- net u6-134: now reaches U6.134
- net u6-135: now reaches U6.135
- net u6-136: now reaches U6.136
- net u6-137: now reaches U6.137
- net u6-138: now reaches U6.138
- net u6-139: now reaches U6.139
- net u6-140: now reaches U6.140
- net u6-141: now reaches U6.141
- net u6-143: now reaches U6.143
- net u6-23: now reaches U6.23
- net u6-43: now reaches U6.43
- net u6-44: now reaches U6.44
- net u6-45: now reaches U6.45
- net u6-46: now reaches U6.46
- net u6-47: now reaches U6.47
- net u6-48: now reaches U6.48
- net u6-49: now reaches U6.49
- net u6-50: now reaches U6.50
- net u6-51: now reaches U6.51
- net u6-52: now reaches U6.52
- net u6-52: now also R53.1
- net u6-53: now reaches U6.53
- net u6-54: now reaches U6.54
- net u6-58: now reaches U6.58
- net u6-59: now reaches U6.59
- net u6-60: now reaches U6.60
- net u6-61: now reaches U6.61
- net u6-86: now reaches U6.86
- net u6-89: now reaches U6.89
- net u6-90: now reaches U6.90
- net u6-93: now reaches U6.93
- net u6-94: now reaches U6.94
- net u6-97: now reaches U6.97
- net u6-98: now reaches U6.98
- net r53-2: now reaches R53.2

Commit message: PCB update
Parts:
- added BT1: Battery_Cell, _mine:286_bat, symbol Device:Battery_Cell
- added C58, C68: 10u, Capacitor_THT:CP_Radial_D5.0mm_P2.50mm, symbol Device:C_Polarized_Small
- added C63: DNP, Capacitor_THT:C_Disc_D3.0mm_W1.6mm_P2.50mm, symbol Device:C_Small
- added C80: ~, Capacitor_THT:C_Disc_D4.3mm_W1.9mm_P5.00mm, symbol Device:C_Small
- added C82: DNP, Capacitor_THT:C_Disc_D4.3mm_W1.9mm_P5.00mm, symbol Device:C_Small
- added D3, D4: D_Small, Diode_THT:D_A-405_P10.16mm_Horizontal, symbol Device:D_Small
- added J11: Bus_ISA_16bit, _mine:ISA_16bit, symbol Connector:Bus_ISA_16bit
- added JP9: Conn_01x04, Connector_PinHeader_2.54mm:PinHeader_1x04_P2.54mm_Vertical, symbol Connector_Generic:Conn_01x04
- added POWER1: Conn_01x12_Pin, Connector_Molex:Molex_KK-396_A-41791-0012_1x12_P3.96mm_Vertical, symbol Connector:Conn_01x12_Pin
- added Q3: 2SA1015, Package_TO_SOT_THT:TO-92_Inline_Wide, symbol Transistor_BJT:2SA1015
- added R45, R46, R47, R49, R55: R_Small, Resistor_THT:R_Axial_DIN0204_L3.6mm_D1.6mm_P5.08mm_Horizontal, symbol Device:R_Small
- added RA5: R_Network04, Resistor_THT:R_Array_SIP5, symbol Device:R_Network04
- added RP2, RP3, RP4, RP5: 10R, Resistor_THT:R_Array_SIP8, symbol Device:R_Pack04_SIP
- added RP6: 40R, Resistor_THT:R_Array_SIP8, symbol Device:R_Pack04_SIP
- added U4: 74LS32, Package_DIP:DIP-14_W7.62mm, symbol 74xx:74LS32
- renumbered U100 to U12
Connections:
- net ra6-5 is gone; now on net j12-io_ready: RA6.5 (R4)
- net u1-1 is gone; now on net u16-2: U1.1 (A->B), U3.1 (A->B)
- net u16-3 is gone; now on an unnamed net: U16.3, U16.5
- net u16-4 is gone; now on an unnamed net: U16.4
- net u16-8 is gone; now on an unnamed net: U16.8
- net u18-2 is gone; now on net u6-71: U18.2 (A0)
- net u18-3 is gone; now on net u15-5: U18.3 (A1)
- net u18-4 is gone; now on net u15-6: U18.4 (A2)
- net u18-5 is gone; now on net u19-15: U18.5 (A3)
- net u18-6 is gone; now on net u19-16: U18.6 (A4)
- net u18-8 is gone; now on net u19-18: U18.8 (A6)
- net u20-15 is gone; now on net u16-1: U20.15 (IO5)
- net x2-1 is gone; now on an unnamed net: X2.1
- net +12V: now also POWER1.10 (Pin_10)
- net -12V: now also POWER1.9 (Pin_9)
- net -5V: now also POWER1.4 (Pin_4)
- net GND: now also POWER1.5 (Pin_5), POWER1.6 (Pin_6), POWER1.7 (Pin_7), POWER1.8 (Pin_8), U4.7 (GND)
- net VDD: now also POWER1.1 (Pin_1), POWER1.11 (Pin_11), POWER1.2 (Pin_2), POWER1.3 (Pin_3), RA5.1 (common), U4.14 (VCC)
- net u19-17: now also U18.7 (A5)
- net u19-19: now also U18.9 (A7)
- net u5-33: now also U20.4 (I4)
- net u6-115: now also C25.2
- net u6-71: now also U19.12 (D0)
- net PW_GOOD: now reaches U16.13
- net PW_GOOD: now also POWER1.12 (Pin_12)
- net j12-io_ready: now reaches J12.41 (IO_READY)
- net at R57.2: now also C60.2, U16.9
- net x2-2: no longer names the net of C60.1, X2.2
Other:
- moved on the sheet: C60, J12, R57, U15, U16A, U16B, U16C, U16D, U6, X2
