File: KiCAD/286.kicad_sch (KiCad schematic)
At the start: 106 parts, among them CON1 Conn_02x20_Odd_Even, CON2 Conn_02x17_Odd_Even, J11 Bus_ISA_16bit, J12 Bus_ISA_16bit, Q3 2SA1015, Q4 2SC1815, U1 74LS245, U12 74LS00, U14 74LS06, U15 HM6818P, U16 4069, U18 74LS245, U19 D8041AHC, U20 PAL16L8, U3 74LS245, U4 74LS32, U5 80C287, U6 ST62C241-A, U7 N80L286-16/S, U8 MCS3201FN, X1 Crystal, X2 Crystal

Commit message: PCB update
Parts:
- added U10: ST62C303-A, Package_QFP:PQFP-160_28x28mm_P0.65mm, symbol _mine_d:ST62C303-A
- KEYBOARD1: footprint (none) -> _mine:286_DIN5
Connections:
- net VDD is gone; now on net +5V: C28.2, JP19.1 (Pin_1), POWER1.1 (Pin_1), POWER1.11 (Pin_11), POWER1.2 (Pin_2), POWER1.3 (Pin_3), R17.2, RA2.1 (common), RA5.1 (common), RP10.1 (common), RP11.1 (common), U1.20 (VCC), U12.14 (VCC), U14.14 (VCC), U18.20 (VCC), U19.26 (VDD), U20.20 (VCC), U3.20 (VCC), U4.14 (VCC), U5.9 (VDD), U6.1, U6.100, U6.120, U6.20, U6.40, U6.81, U7.30 (VCC), U7.62 (VCC)
- net con1-23 is gone; now on net u8-24: CON1.23 (Pin_23)
- net con1-31 is gone; now on net jp15-2: CON1.31 (Pin_31)
- net con1-37 is gone; now on net u20-17: CON1.37 (Pin_37)
- net j12-ba6 is gone; now on net BA06: J12.56 (BA06)
- net j12-ba7 is gone; now on net BA07: J12.55 (BA07)
- net ra7-9 is gone; now on net KB_DATA: C76.1, RA7.9 (R8)
- net rp1-10 is gone; now on net jp14-2: RP1.10 (R9)
- net rp1-2 is gone; now on net jp10-2: RP1.2 (R1)
- net rp1-6 is gone; now on net u8-29: RP1.6 (R5)
- net rp8-2 is gone; now on net u8-24: RP8.2 (R1.2)
- net rp8-4 is gone; now on net j12-ior: RP8.4 (R2.2)
- net u100-1 is gone; now on net u6-39: U12.1, U12.2
- net u100-3 is gone; now on net u19-reset: U12.3
- net u100-4 is gone; now on net u15-19: U12.4, U12.5
- net u14-13 is gone; now on net u6-39: U14.13
- net u14-5 is gone; now on net u19-37: U14.5
- net u14-6 is gone; now on net KB_CLK: U14.6
- net u16-1 is gone; now on net j12-ior: U16.1, U20.15 (IO5)
- net u18-11 is gone; now on net DB7: U18.11 (B7)
- net u18-12 is gone; now on net DB6: U18.12 (B6)
- net u18-13 is gone; now on net DB5: U18.13 (B5)
- net u18-14 is gone; now on net DB4: U18.14 (B4)
- net u18-15 is gone; now on net DB3: U18.15 (B3)
- net u18-16 is gone; now on net DB2: U18.16 (B2)
- net u18-17 is gone; now on net DB1: U18.17 (B1)
- net u18-18 is gone; now on net DB0: U18.18 (B0)
- net u19-9 is gone; now on net BA02: U19.9 (A0)
- net u20-14 is gone; now on net jp14-2: U20.14 (IO6)
- net u20-2 is gone; now on net BA02: U20.2 (I2)
- net u20-3 is gone; now on net BA03: U20.3 (I3)
- net u20-8 is gone; now on net BA08: U20.8 (I8), U8.9 (SA8)
- net u5-33 is gone; now on net BA04: U20.4 (I4), U5.33
- net u6-54 is gone; now on net j12-io_ready: U6.54
- net u6-61 is gone; now on net jp1-3: RA2.2 (R1), U6.61
- net u8-10 is gone; now on net BA09: U8.10 (SA9)
- net u8-2 is gone; now on net con1-33: U8.2 (SA1)
- net u8-25 is gone; now on net j12-ior: U8.25 (~{IOR})
- net u8-26 is gone; now on net j12-irq6: U8.26 (IRQ)
- net u8-28 is gone; now on net j12-tc: U8.28 (T/C)
- net u8-3 is gone; now on net BA02: U8.3 (SA2)
- net u8-4 is gone; now on net BA03: U8.4 (SA3)
- net u8-5 is gone; now on net BA04: U8.5 (SA4)
- net u8-6 is gone; now on net BA05: U8.6 (SA5)
- net u8-66 is gone; now on net con2-34: RP1.5 (R4), U8.66 (~{DSKCHNG})
- net u8-7 is gone; now on net BA06: U8.7 (SA6)
- net u8-8 is gone; now on net BA07: U8.8 (SA7)
- net A1: now also U10.34
- net A10: now also U10.14
- net A11: now also U10.13
- net A12: now also U10.11
- net A13: now also U10.10
- net A14: now also U10.9
- net A15: now also U10.3
- net A16: now also U10.1
- net A2: now also U10.33
- net A3: now also U10.27
- net A4: now also U10.26
- net A5: now also U10.25
- net A6: now also U10.23
- net A7: now also U10.22
- net A8: now also U10.21
- net A9: now also U10.15
- net D10: now also U5.12
- net D11: now also U5.11
- net D12: now also U5.8
- net D13: now also U5.7
- net D15: now also U5.5
- net D8: now also U5.15
- net D9: now also U5.14
- net GND: now also BT1.2 (-), C30.1, C31.1, C38.2, C40.1, C43.1, C44.1, C45.1, C50.1, C58.1, C62.1, C7.2, C76.2, C77.2, CON1.19 (Pin_19), CON1.2 (Pin_2), CON1.22 (Pin_22), CON1.24 (Pin_24), CON1.26 (Pin_26), CON1.30 (Pin_30), CON1.40 (Pin_40), CON2.1 (Pin_1), CON2.11 (Pin_11), CON2.13 (Pin_13), CON2.15 (Pin_15), CON2.17 (Pin_17), CON2.19 (Pin_19), CON2.21 (Pin_21), CON2.23 (Pin_23), CON2.25 (Pin_25), CON2.27 (Pin_27), CON2.29 (Pin_29), CON2.3 (Pin_3), CON2.31 (Pin_31), CON2.33 (Pin_33), CON2.5 (Pin_5), CON2.7 (Pin_7), CON2.9 (Pin_9), J12.1 (GND), J12.31 (GND), JP10.1 (Pin_1), JP14.1 (Pin_1), JP5.1 (Pin_1), JP9.3 (Pin_3), JP9.4 (Pin_4), KEYBOARD1.2, R46.1, U15.12 (VSS), U18.19 (CE), U8.16 (VSS), U8.31 (VSS), U8.35 (I7), U8.36 (I6), U8.37 (I5), U8.38 (I4), U8.39 (I3), U8.40 (I2), U8.41 (I1), U8.42 (I0), U8.45 (VSS), U8.50 (VSS), U8.54 (VSS), U8.57 (VSS), U8.60 (VSS), U8.67 (VSS), U8.68 (VSS), U10.109, U10.120, U10.18, U10.30, U10.40, U10.43, U10.50, U10.55, U10.6, U10.80; no longer U5.39 (VSS)
- net VBAT: now also C58.2, Q3.2 (C), R48.1
- net c62-2: now also U15.18 (~{RESET}), U15.22 (PS)
- net con1-33: now also U20.1 (I1), U5.29, U10.107
- net con1-35: now also U20.13 (IO7)
- net con1-5: now also U1.8 (A6)
- net con1-7: now also U1.7 (A5)
- net j12-dack0: now also U10.98
- net j12-drq1: now also U10.93
- net j12-io: now also U10.37
- net j12-io_ready: now also U10.36
- net j12-iocs16: now also CON1.32 (Pin_32), U4.2
- net j12-irq4: now also U10.89
- net jp1-1: now also U19.29 (P12)
- net jp1-3: now also U14.12, U14.4
- net jp15-1: now also U10.82
- net jp2-1: now also U14.3
- net jp20-2: now also U5.32
- net pr11-3: now also U10.115
- net ra2-5: now also U5.25, U10.104
- net u1-19: now also U4.5
- net u1-2: now also CON1.17 (Pin_17)
- net u1-3: now also CON1.15 (Pin_15)
- net u15-5: now also U10.73
- net u15-6: now also U10.72
- net u16-10: now also U14.9
- net u16-11: now also U19.38 (P27/~{DACK})
- net u16-12: now also U15.13 (~{CE})
- net u16-2: now also U4.4
- net u19-10: now also U5.28
- net u19-15: now also U10.71
- net u19-16: now also U10.70
- net u19-17: now also U10.69
- net u19-18: now also U10.68
- net u19-19: now also U15.11 (AD7), U10.67
- net u19-6: now also U10.46
- net u19-8: now also U5.27
- net u20-18: now also CON1.38 (Pin_38)
- net u3-19: now also U4.3
- net u6-123: now also U10.57
- net u6-148: now also U10.2
- net u6-43: now also U10.117
- net u6-44: now also U10.116
- net u6-46: now also U10.114
- net u6-47: now also U10.113
- net u6-48: now also U10.112
- net u6-49: now also U10.101
- net u6-50: now also U10.100
- net u6-51: now also U10.99
- net u6-52: now also U10.59
- net u6-53: now also C7.1, RA7.7 (R6), U14.10, U15.16 (~{STBY})
- net u6-58: now also RA6.2 (R1), U14.1, U19.2 (XTAL1)
- net u6-71: now also U15.4 (AD0), U10.74
- net u8-1: now also U10.108
- net u8-23: now also U10.91
- net u8-27: now also U10.97
- net u8-48: now also CON2.16 (Pin_16)
- net u8-49: now also CON2.10 (Pin_10)
- net u8-51: now also CON2.12 (Pin_12)
- net u8-53: now also CON2.24 (Pin_24)
- net u8-55: now also CON2.18 (Pin_18)
- net u8-58: now also CON2.2 (Pin_2)
- net x1-1: now also U10.41
- net x1-2: now also R44.2, U10.42
- net ~{READY}: now also RA6.4 (R3)
- net +5V: now reaches C44.2
- net +5V: now also C30.2, C31.2, C38.1, C40.2, C43.2, C45.2, D1.1 (K), D4.2 (A), KEYBOARD1.4, Q3.1 (E), R45.1, RA6.1 (common), RA7.1 (common), RP1.1 (common), U19.25 (PROG), U19.40 (VCC), U8.17 (VDD), U8.32 (VDD), U10.102, U10.118, U10.12, U10.24, U10.49, U10.66, U10.83, U10.84
- net bat+: now reaches BT1.1 (+)
- net bat+: now also D2.2 (A), D3.1 (K), R49.2
- net d3-2: now reaches JP9.1 (Pin_1)
- net d3-2: now also D3.2 (A)
- net r46-2: now reaches R46.2
- net r46-2: now also R45.2
- net DB0: now reaches U8.12 (SD0)
- net DB0: now also J12.40 (DB0), U1.18 (B0)
- net DB1: now reaches U8.13 (SD1)
- net DB1: now also J12.39 (DB1), U1.17 (B1)
- net DB2: now reaches U8.14 (SD2)
- net DB2: now also J12.38 (DB2), U1.16 (B2)
- net DB3: now reaches U8.15 (SD3)
- net DB3: now also J12.37 (DB3), U1.15 (B3)
- net DB4: now reaches U8.18 (SD4)
- net DB4: now also J12.36 (DB4), U1.14 (B4)
- net DB5: now reaches U8.19 (SD5)
- net DB5: now also J12.35 (DB5), U1.13 (B5)
- net DB6: now reaches U8.20 (SD6)
- net DB6: now also J12.34 (DB6), U1.12 (B6)
- net DB7: now reaches U8.21 (SD7)
- net DB7: now also J12.33 (DB7)
- net u8-22: now reaches U8.22 (RESET)
- net u8-22: now also C50.2, R2.1
- net u8-29: now reaches U8.29 (ADDSEL)
- net u8-29: now also JP5.2 (Pin_2)
- net jp10-2: now reaches U8.30 (~{CS})
- net jp10-2: now also JP10.2 (Pin_2)
- net u8-52: now reaches U8.52 (~{DS0})
- net u8-52: now also CON2.14 (Pin_14)
- net u8-56: now reaches U8.56 (~{HEAD})
- net u8-56: now also CON2.32 (Pin_32)
- net d4-2: now reaches D4.1 (K)
- net d4-2: now also R49.1
- net j12-drq3: now reaches J12.16 (DRQ3)
- net j12-drq3: now also U10.92
- net j12-irq7: now reaches J12.21 (IRQ7)
- net j12-irq7: now also U10.86
- net j12-irq6: now reaches J12.22 (IRQ6)
- net j12-irq6: now also U10.87
- net j12-tc: now reaches J12.27 (TC)
- net j12-tc: now also U10.52
- net j12-ale: now reaches J12.28 (ALE)
- net j12-ale: now also CON1.28 (Pin_28), RA7.5 (R4)
- net j12-osc: now reaches J12.30 (OSC)
- net j12-irq2: now reaches J12.4 (IRQ2)
- net j12-irq2: now also U10.76
- net BA09: now reaches J12.53 (BA09)
- net BA09: now also U10.32
- net BA08: now reaches J12.54 (BA08)
- net BA08: now also U10.38
- net BA05: now reaches J12.57 (BA05)
- net BA03: now reaches J12.59 (BA03)
- net BA02: now reaches J12.60 (BA02)
- net BA02: now also CON1.36 (Pin_36), U5.31, U10.56
- net j12-sbhe: now reaches J12.81 (SBHE)
- net j12-sbhe: now also U10.110
- net j12-la23: now reaches J12.82 (LA23)
- net j12-la23: now also U10.111
- net u12-13: now reaches U12.13
- net u1-4: now reaches U1.4 (A2)
- net u1-4: now also CON1.13 (Pin_13)
- net r47-1: now reaches R47.1
- net q3-3: now reaches R47.2
- net q3-3: now also Q3.3 (B)
- net u12-6: now reaches U12.6
- net u12-6: now also U10.75
- net u5-39: now reaches JP19.2 (Pin_2)
- net u5-39: now also U5.39 (VSS)
- net rp11-5: now reaches RP11.5 (R4)
- net rp11-5: now also U10.119
- net u15-14: now reaches U15.14 (AS)
- net u15-14: now also U10.47
- net u15-15: now reaches U15.15 (R/~{W})
- net u15-15: now also U10.48
- net u15-17: now reaches U15.17 (DS)
- net u15-17: now also U10.51
- net u15-19: now reaches U15.19 (~{IRQ})
- net u15-19: now also RA7.3 (R2)
- net u20-16: now reaches U20.16 (IO4)
- net BA06: now reaches U20.6 (I6)
- net BA07: now reaches U20.7 (I7)
- net BA07: now also U10.39
- net u19-reset: now reaches CON1.1 (Pin_1)
- net u19-reset: now also RA7.4 (R3), U19.4 (~{RESET})
- net con1-3: now reaches CON1.3 (Pin_3)
- net con1-39: now reaches CON1.39 (Pin_39)
- net jp14-2: now reaches JP14.2 (Pin_2)
- net KB_CLK: now reaches U19.1 (TEST0)
- net KB_CLK: now also C77.1, KEYBOARD1.1, RA7.2 (R1)
- net jp7-3: now reaches U19.23 (P22)
- net jp7-3: now also JP7.3 (Pin_3)
- net jp2-2: now reaches U19.27 (P10)
- net jp2-2: now also JP2.2 (Pin_2)
- net u19-3: now reaches U19.3 (XTAL2)
- net u19-3: now also RA6.3 (R2), U14.2
- net u19-31: now reaches U19.31 (P14)
- net u19-31: now also RA7.6 (R5)
- net jp7-1: now reaches U19.32 (P15)
- net jp7-1: now also JP7.1 (Pin_1)
- net u19-33: now reaches U19.33 (P16)
- net u19-33: now also RA7.8 (R7)
- net u19-35: now reaches U19.35 (P24/OBF)
- net u19-35: now also U10.85
- net u19-37: now reaches U19.37 (P26/DRQ)
- net KB_DATA: now reaches U19.39 (TEST1)
- net KB_DATA: now also KEYBOARD1.3, U14.8
- net jp15-2: now reaches JP15.2 (Pin_2)
- net u10-5: now reaches RP8.1 (R1.1)
- net u10-5: now also U10.5
- net u10-8: now reaches RP8.3 (R2.1)
- net u10-8: now also U10.8
- net u5-26: now reaches U5.26
- net u5-26: now also U10.103
- net u5-34: now reaches U5.34
- net u5-35: now reaches U5.35
- net u5-35: now also U10.105
- net j12-ba10 renamed BA10
- net BA10: now also U10.31
- net j12-ba11 renamed BA11
- net BA11: now also U10.29
- net j12-ba12 renamed BA12
- net BA12: now also U10.28
- net j12-ba13 renamed BA13
- net BA13: now also U10.20
- net j12-ba14 renamed BA14
- net BA14: now also U10.19
- net j12-ba4 renamed BA04
- net BA04: now also U10.53
- new net u10-16: U10.16
- new net u10-17: U10.17
- new net u10-35: U10.35
- new net u10-4: U10.4
- new net u10-44: U10.44
- new net u10-45: U10.45
- new net u10-54: U10.54
- new net u10-58: U10.58
- new net u10-60: U10.60
- new net u10-61: U10.61
- new net u10-62: U10.62
- new net u10-63: U10.63
- new net u10-64: U10.64
- new net u10-65: U10.65
- new net u10-7: U10.7
- new net u10-77: U10.77
- new net u10-78: U10.78
- new net u10-79: U10.79
- new net u10-81: U10.81
- new net u10-88: U10.88
- new net u10-90: U10.90
- new net u10-94: U10.94
- new net u10-95: U10.95
- new net u10-96: U10.96
- no-connect marks 5 -> 35
Other:
- moved on the sheet: CON2, J11, J12, KEYBOARD1
