File: KiCAD/286.kicad_sch (KiCad schematic)
At the start: 107 parts, among them CON1 Conn_02x20_Odd_Even, CON2 Conn_02x17_Odd_Even, J11 Bus_ISA_16bit, J12 Bus_ISA_16bit, Q3 2SA1015, Q4 2SC1815, U1 74LS245, U10 ST62C303-A, U12 74LS00, U14 74LS06, U15 HM6818P, U16 4069, U18 74LS245, U19 D8041AHC, U20 PAL16L8, U3 74LS245, U4 74LS32, U5 80C287, U6 ST62C241-A, U7 N80L286-16/S, U8 MCS3201FN, X1 Crystal, X2 Crystal

Commit message: PCB update
Parts:
- added DL1: 31A-5500, _mine:31A-5500, symbol _mine_d:31A-5500
- added J10, J9: Bus_ISA_16bit, _mine:ISA_16bit, symbol Connector:Bus_ISA_16bit
- added J17, SPEAKER1: Conn_01x04, Connector_PinHeader_2.54mm:PinHeader_1x04_P2.54mm_Vertical, symbol Connector_Generic:Conn_01x04
- added KEYLOCK1: Conn_01x05, Connector_PinHeader_2.54mm:PinHeader_1x05_P2.54mm_Vertical, symbol Connector_Generic:Conn_01x05
- added Q1, Q2: 2SC1815, Package_TO_SOT_THT:TO-92_Inline_Wide, symbol Transistor_BJT:2SC1815
- added R10: R_Small, Resistor_THT:R_Axial_DIN0204_L3.6mm_D1.6mm_P5.08mm_Horizontal, symbol Device:R_Small
- added R52: R_Small, _mine:R_Axial_L3.6mm_D1.6mm_P4.5mm_Horizontal, symbol Device:R_Small
- added RA3: R_Network08, Resistor_THT:R_Array_SIP9, symbol Device:R_Network08
- added RESET1, TUR-LED1, TURBO1: Conn_01x02, Connector_PinSocket_2.54mm:PinSocket_1x02_P2.54mm_Vertical, symbol Connector_Generic:Conn_01x02
- added U11: 74LS245, Package_DIP:DIP-20_W7.62mm, symbol 74xx:74LS245
- added U17: 74AHCT125, Package_DIP:DIP-14_W7.62mm, symbol 74xx:74AHCT125
Connections:
- net con1-33 is gone; now on net BA01: CON1.33 (Pin_33), U10.107, U20.1 (I1), U5.29, U8.2 (SA1)
- net con1-35 is gone; now on net BA00: CON1.35 (Pin_35), U20.13 (IO7)
- net j12-la23 is gone; now on net LA23: J12.82 (LA23), U10.111
- net r53-2 is gone; now on net j12-refresh: R53.2
- net rp8-6 is gone; now on net j12-memw: RP10.5 (R4), RP8.6 (R3.2)
- net u1-19 is gone; now on net u20-16: U1.19 (CE), U4.5
- net u10-16 is gone; now on net BA16: U10.16
- net u10-17 is gone; now on net BA15: U10.17
- net u10-4 is gone; now on net BA18: U10.4
- net u10-44 is gone; now on net BA06: U10.44
- net u10-45 is gone; now on net BA05: U10.45
- net u10-54 is gone; now on net BA03: U10.54
- net u10-58 is gone; now on net j12-master: U10.58
- net u10-60 is gone; now on net j12-dack5: U10.60
- net u10-61 is gone; now on net j12-dack6: U10.61
- net u10-62 is gone; now on net j12-dack7: U10.62
- net u10-63 is gone; now on net j12-drq5: U10.63
- net u10-64 is gone; now on net j12-drq6: U10.64
- net u10-65 is gone; now on net j12-drq7: U10.65
- net u10-7 is gone; now on net BA17: U10.7
- net u10-77 is gone; now on net j12-irq10: U10.77
- net u10-78 is gone; now on net j12-irq11: U10.78
- net u10-79 is gone; now on net j12-irq12: U10.79
- net u10-81 is gone; now on net j12-irq15: U10.81
- net u10-88 is gone; now on net j12-irq5: U10.88
- net u10-90 is gone; now on net j12-irq3: U10.90
- net u10-94 is gone; now on net j12-drq0: U10.94
- net u10-95 is gone; now on net j12-dack3: U10.95
- net u10-96 is gone; now on net j12-dack1: U10.96
- net u19-10 is gone; now on net u6-34: U19.10 (~{WR}), U5.28
- net u20-17 is gone; now on net u4-1: CON1.37 (Pin_37), U20.17 (I03)
- net u20-5 is gone; now on net BA05: U20.5 (I5)
- net u20-9 is gone; now on net BA09: U20.9 (I9)
- net u3-11 is gone; now on net j12-d8: U3.11 (B7)
- net u3-12 is gone; now on net j12-d9: U3.12 (B6)
- net u3-16 is gone; now on net j12-d13: U3.16 (B2)
- net u3-18 is gone; now on net j12-d15: J12.98 (D15), U3.18 (B0)
- net u6-123 is gone; now on net j12-osc: U10.57, U6.123
- net u6-32 is gone; now on net j12-ale: U6.32
- net u6-39 is gone; now on net j12-reset: R2.2, U12.1, U12.2, U14.13, U6.39
- net u6-43 is gone; now on net j12-clk: U10.117, U6.43
- net u6-55 is gone; now on net j12-unused: U6.55
- net u8-1 is gone; now on net BA00: U10.108, U8.1 (SA0)
- net u8-11 is gone; now on net j12-aen: U8.11 (AEN)
- net u8-23 is gone; now on net j12-drq2: U10.91, U8.23 (DRQ)
- net u8-24 is gone; now on net j12-iow: CON1.23 (Pin_23), RP8.2 (R1.2), U8.24 (~{IOW})
- net u8-27 is gone; now on net j12-dack2: U10.97, U8.27 (~{DACK})
- net +12V: now also J11.9 (+12V), J10.9 (+12V), J9.9 (+12V)
- net +5V: now also C63.1, C80.2, J11.29 (VCC), J11.3 (+5V), J11.78 (+5V), J12.29 (VCC), J12.3 (+5V), J12.78 (+5V), U10.127, U10.134, U10.142, U10.148, U10.160, DL1.14 (VCC), J10.29 (VCC), J10.3 (+5V), J10.78 (+5V), J9.29 (VCC), J9.3 (+5V), J9.78 (+5V), R52.1, RA3.1 (common), SPEAKER1.4 (Pin_4), U11.20 (VCC), U17.14 (VCC)
- net -12V: now also J11.7 (-12V), J10.7 (-12V), J9.7 (-12V)
- net -5V: now also J11.5 (-5V), J10.5 (-5V), J9.5 (-5V)
- net A17: now also U10.159
- net A18: now also U10.158
- net A19: now also U10.157
- net A21: now also U10.151
- net A22: now also U10.150
- net A23: now also U10.149
- net BA02: now also J11.60 (BA02), J10.60 (BA02), J9.60 (BA02)
- net BA03: now also J11.59 (BA03), J10.59 (BA03), J9.59 (BA03)
- net BA04: now also J11.58 (BA04), J10.58 (BA04), J9.58 (BA04)
- net BA05: now also J11.57 (BA05), J10.57 (BA05), J9.57 (BA05)
- net BA06: now also J11.56 (BA06), J10.56 (BA06), J9.56 (BA06)
- net BA07: now also J11.55 (BA07), J10.55 (BA07), J9.55 (BA07)
- net BA08: now also J11.54 (BA08), J10.54 (BA08), J9.54 (BA08)
- net BA09: now also J11.53 (BA09), J10.53 (BA09), J9.53 (BA09)
- net BA10: now also J11.52 (BA10), J10.52 (BA10), J9.52 (BA10)
- net BA11: now also J11.51 (BA11), J10.51 (BA11), J9.51 (BA11)
- net BA12: now also J11.50 (BA12), J10.50 (BA12), J9.50 (BA12)
- net BA13: now also J11.49 (BA13), J10.49 (BA13), J9.49 (BA13)
- net BA14: now also J11.48 (BA14), J10.48 (BA14), J9.48 (BA14)
- net DB0: now also J11.40 (DB0), J10.40 (DB0), J9.40 (DB0)
- net DB1: now also J11.39 (DB1), J10.39 (DB1), J9.39 (DB1)
- net DB2: now also J11.38 (DB2), J10.38 (DB2), J9.38 (DB2)
- net DB3: now also J11.37 (DB3), J10.37 (DB3), J9.37 (DB3)
- net DB4: now also J11.36 (DB4), J10.36 (DB4), J9.36 (DB4)
- net DB5: now also J11.35 (DB5), J10.35 (DB5), J9.35 (DB5)
- net DB6: now also J11.34 (DB6), J10.34 (DB6), J9.34 (DB6)
- net DB7: now also J11.33 (DB7), J10.33 (DB7), J9.33 (DB7), U17.2, U17.6
- net GND: now also C58.2, C63.2, C80.1, C82.1, J11.1 (GND), J11.10 (GND), J11.31 (GND), J11.80 (GND), J12.10 (GND), J12.80 (GND), U10.128, U10.141, U10.154, DL1.7 (GND), J10.1 (GND), J10.10 (GND), J10.31 (GND), J10.80 (GND), J9.1 (GND), J9.10 (GND), J9.31 (GND), J9.80 (GND), KEYLOCK1.3 (Pin_3), KEYLOCK1.5 (Pin_5), Q1.1 (E), Q2.1 (E), RESET1.1 (Pin_1), SPEAKER1.3 (Pin_3), TURBO1.1 (Pin_1), U11.10 (GND), U11.19 (CE), U17.7 (GND); no longer C58.1
- net INTR: now also U10.146
- net NMI: now also U10.147
- net VBAT: now also C58.1; no longer C58.2
- net bk2-2: now also RP2.7 (R4.1)
- net bk4-1: now also RP6.4 (R2.2)
- net bk4-2: now also RP6.7 (R4.1)
- net con1-3: now also U17.3, U17.5
- net j12-aen: now also J11.42 (AEN), U10.152, J10.42 (AEN), J9.42 (AEN)
- net j12-ale: now also J11.28 (ALE), U10.135, J10.28 (ALE), J9.28 (ALE)
- net j12-dack0: now also J11.70 (~{DACK0}), J10.70 (~{DACK0}), J9.70 (~{DACK0})
- net j12-drq1: now also J11.18 (DRQ1), J10.18 (DRQ1), J9.18 (DRQ1)
- net j12-drq3: now also J11.16 (DRQ3), J10.16 (DRQ3), J9.16 (DRQ3)
- net j12-io: now also J11.32 (IO), J10.32 (IO), J9.32 (IO)
- net j12-io_ready: now also J11.41 (IO_READY), J10.41 (IO_READY), J9.41 (IO_READY)
- net j12-iocs16: now also J11.64 (~{IOCS16}), RA5.4 (R3), J10.64 (~{IOCS16}), J9.64 (~{IOCS16})
- net j12-ior: now also J11.14 (~{IOR}), J10.14 (~{IOR}), J9.14 (~{IOR})
- net j12-irq2: now also J11.4 (IRQ2), J10.4 (IRQ2), J9.4 (IRQ2)
- net j12-irq4: now also J11.24 (IRQ4), J10.24 (IRQ4), J9.24 (IRQ4)
- net j12-irq6: now also J11.22 (IRQ6), J10.22 (IRQ6), J9.22 (IRQ6)
- net j12-irq7: now also J11.21 (IRQ7), J10.21 (IRQ7), J9.21 (IRQ7)
- net j12-master: now also J11.79 (MASTER), RA5.2 (R1), J10.79 (MASTER), J9.79 (MASTER)
- net j12-memcs16: now also J11.63 (~{MEMCS16}), RA5.5 (R4), J10.63 (~{MEMCS16}), J9.63 (~{MEMCS16})
- net j12-memr: now also J11.89 (~{MEMR}), RP8.7 (R4.1), J10.89 (~{MEMR}), J9.89 (~{MEMR})
- net j12-osc: now also J11.30 (OSC), J10.30 (OSC), J9.30 (OSC)
- net j12-sbhe: now also J11.81 (SBHE), J10.81 (SBHE), J9.81 (SBHE)
- net j12-tc: now also J11.27 (TC), J10.27 (TC), J9.27 (TC)
- net jp15-1: now also J11.69 (IRQ14), J12.69 (IRQ14), J10.69 (IRQ14), J9.69 (IRQ14)
- net u10-35: now also R10.1
- net u12-13: now also U10.145
- net u19-34: now also KEYLOCK1.4 (Pin_4)
- net u20-19: now also U17.4
- net u5-34: now also U10.138
- net u6-129: now also DL1.12 (1)
- net u6-130: now also DL1.10 (3)
- net u6-131: now also DL1.8 (OUT)
- net u6-135: now also RP4.2 (R1.2)
- net u6-140: now also RP3.6 (R3.2)
- net u6-141: now also RP3.8 (R4.2)
- net u6-23: now also RP11.2 (R1)
- net u6-30: now also U10.137
- net u6-31: now also U10.136
- net u6-33: now also U10.133
- net u6-34: now also U10.132
- net u6-35: now also U10.131
- net u6-36: now also U10.124
- net u6-37: now also U10.123
- net u6-38: now also U10.122
- net u6-78: now also U11.2 (A0)
- net u6-82: now also U11.1 (A->B)
- net u6-86: now also U11.3 (A1)
- net u6-90: now also U11.4 (A2)
- net u6-94: now also U11.5 (A3)
- net ~{ERROR}: now also RP11.4 (R3)
- net j12-smemw: now reaches J12.11 (~{SMEMW})
- net j12-smemw: now also J11.11 (~{SMEMW}), J10.11 (~{SMEMW}), J9.11 (~{SMEMW})
- net j12-smemr: now reaches J12.12 (~{SMEMR})
- net j12-smemr: now also J11.12 (~{SMEMR}), R55.2, J10.12 (~{SMEMR}), J9.12 (~{SMEMR})
- net j12-iow: now reaches J12.13 (~{IOW})
- net j12-iow: now also J11.13 (~{IOW}), J10.13 (~{IOW}), J9.13 (~{IOW})
- net j12-dack3: now reaches J12.15 (~{DACK3})
- net j12-dack3: now also J11.15 (~{DACK3}), J10.15 (~{DACK3}), J9.15 (~{DACK3})
- net j12-dack1: now reaches J12.17 (~{DACK1})
- net j12-dack1: now also J11.17 (~{DACK1}), J10.17 (~{DACK1}), J9.17 (~{DACK1})
- net j12-refresh: now reaches J12.19 (~{REFRESH})
- net j12-refresh: now also J11.19 (~{REFRESH}), J10.19 (~{REFRESH}), J9.19 (~{REFRESH}), R52.2
- net j12-reset: now reaches J12.2 (RESET)
- net j12-reset: now also C82.2, J11.2 (RESET), U10.121, J10.2 (RESET), J9.2 (RESET)
- net j12-clk: now reaches J12.20 (CLK)
- net j12-clk: now also J11.20 (CLK), J10.20 (CLK), J9.20 (CLK)
- net j12-irq5: now reaches J12.23 (IRQ5)
- net j12-irq5: now also J11.23 (IRQ5), J10.23 (IRQ5), J9.23 (IRQ5)
- net j12-irq3: now reaches J12.25 (IRQ3)
- net j12-irq3: now also J11.25 (IRQ3), J10.25 (IRQ3), J9.25 (IRQ3)
- net j12-dack2: now reaches J12.26 (~{DACK2})
- net j12-dack2: now also J11.26 (~{DACK2}), J10.26 (~{DACK2}), J9.26 (~{DACK2})
- net BA19: now reaches J12.43 (BA19)
- net BA19: now also J11.43 (BA19), U10.156, J10.43 (BA19), J9.43 (BA19)
- net BA18: now reaches J12.44 (BA18)
- net BA18: now also J11.44 (BA18), J10.44 (BA18), J9.44 (BA18)
- net BA17: now reaches J12.45 (BA17)
- net BA17: now also J11.45 (BA17), J10.45 (BA17), J9.45 (BA17)
- net BA16: now reaches J12.46 (BA16)
- net BA16: now also J11.46 (BA16), J10.46 (BA16), J9.46 (BA16)
- net BA15: now reaches J12.47 (BA15)
- net BA15: now also J11.47 (BA15), J10.47 (BA15), J9.47 (BA15)
- net j12-drq2: now reaches J12.6 (DRQ2)
- net j12-drq2: now also J11.6 (DRQ2), J10.6 (DRQ2), J9.6 (DRQ2)
- net BA01: now reaches J12.61 (BA01)
- net BA01: now also J11.61 (BA01), J10.61 (BA01), J9.61 (BA01)
- net BA00: now reaches J12.62 (BA00)
- net BA00: now also J11.62 (BA00), J10.62 (BA00), J9.62 (BA00)
- net j12-irq10: now reaches J12.65 (IRQ10)
- net j12-irq10: now also J11.65 (IRQ10), J10.65 (IRQ10), J9.65 (IRQ10)
- net j12-irq11: now reaches J12.66 (IRQ11)
- net j12-irq11: now also J11.66 (IRQ11), J10.66 (IRQ11), J9.66 (IRQ11)
- net j12-irq12: now reaches J12.67 (IRQ12)
- net j12-irq12: now also J11.67 (IRQ12), J10.67 (IRQ12), J9.67 (IRQ12)
- net j12-irq15: now reaches J12.68 (IRQ15)
- net j12-irq15: now also J11.68 (IRQ15), J10.68 (IRQ15), J9.68 (IRQ15)
- net j12-drq0: now reaches J12.71 (DRQ0)
- net j12-drq0: now also J11.71 (DRQ0), J10.71 (DRQ0), J9.71 (DRQ0)
- net j12-dack5: now reaches J12.72 (~{DACK5})
- net j12-dack5: now also J11.72 (~{DACK5}), J10.72 (~{DACK5}), J9.72 (~{DACK5})
- net j12-drq5: now reaches J12.73 (DRQ5)
- net j12-drq5: now also J11.73 (DRQ5), J10.73 (DRQ5), J9.73 (DRQ5)
- net j12-dack6: now reaches J12.74 (~{DACK6})
- net j12-dack6: now also J11.74 (~{DACK6}), J10.74 (~{DACK6}), J9.74 (~{DACK6})
- net j12-drq6: now reaches J12.75 (DRQ6)
- net j12-drq6: now also J11.75 (DRQ6), J10.75 (DRQ6), J9.75 (DRQ6)
- net j12-dack7: now reaches J12.76 (~{DACK7})
- net j12-dack7: now also J11.76 (~{DACK7}), J10.76 (~{DACK7}), J9.76 (~{DACK7})
- net j12-drq7: now reaches J12.77 (DRQ7)
- net j12-drq7: now also J11.77 (DRQ7), J10.77 (DRQ7), J9.77 (DRQ7)
- net j12-unused: now reaches J12.8 (UNUSED)
- net j12-unused: now also J11.8 (UNUSED), RA5.3 (R2), J10.8 (UNUSED), J9.8 (UNUSED)
- net LA22: now reaches J12.83 (LA22)
- net LA22: now also J11.83 (LA22), U10.125, J10.83 (LA22), J9.83 (LA22)
- net LA21: now reaches J12.84 (LA21)
- net LA21: now also J11.84 (LA21), U10.126, J10.84 (LA21), J9.84 (LA21)
- net LA20: now reaches J12.85 (LA20)
- net LA20: now also J11.85 (LA20), U10.129, J10.85 (LA20), J9.85 (LA20)
- net LA19: now reaches J12.86 (LA19)
- net LA19: now also J11.86 (LA19), U10.130, J10.86 (LA19), J9.86 (LA19)
- net LA18: now reaches J12.87 (LA18)
- net LA18: now also J11.87 (LA18), U10.139, J10.87 (LA18), J9.87 (LA18)
- net LA17: now reaches J12.88 (LA17)
- net LA17: now also J11.88 (LA17), U10.140, J10.88 (LA17), J9.88 (LA17)
- net j12-memw: now reaches J12.90 (~{MEMW})
- net j12-memw: now also J11.90 (~{MEMW}), J10.90 (~{MEMW}), J9.90 (~{MEMW})
- net j12-d8: now reaches J12.91 (D8)
- net j12-d8: now also J11.91 (D8), J10.91 (D8), J9.91 (D8), RA3.5 (R4), U11.11 (B7)
- net j12-d9: now reaches J12.92 (D9)
- net j12-d9: now also J11.92 (D9), J10.92 (D9), J9.92 (D9), RA3.4 (R3), U11.12 (B6)
- net j12-d10: now reaches J12.93 (D10)
- net j12-d10: now also J11.93 (D10), U3.13 (B5), J10.93 (D10), J9.93 (D10), RA3.3 (R2), U11.13 (B5)
- net j12-d11: now reaches J12.94 (D11)
- net j12-d11: now also J11.94 (D11), U3.14 (B4), J10.94 (D11), J9.94 (D11), RA3.2 (R1), U11.14 (B4)
- net j12-d12: now reaches J12.95 (D12)
- net j12-d12: now also J11.95 (D12), U3.15 (B3), J10.95 (D12), J9.95 (D12), RA3.9 (R8), U11.15 (B3)
- net j12-d13: now reaches J12.96 (D13)
- net j12-d13: now also J11.96 (D13), J10.96 (D13), J9.96 (D13), RA3.8 (R7), U11.16 (B2)
- net j12-d14: now reaches J12.97 (D14)
- net j12-d14: now also J11.97 (D14), U3.17 (B1), J10.97 (D14), J9.97 (D14), RA3.7 (R6), U11.17 (B1)
- net LA23: now reaches J11.82 (LA23)
- net LA23: now also J10.82 (LA23), J9.82 (LA23)
- net j12-d15: now reaches J11.98 (D15)
- net j12-d15: now also J10.98 (D15), J9.98 (D15), RA3.6 (R5), U11.18 (B0)
- net u10-155: now reaches R55.1
- net u10-155: now also U10.155
- net u4-6: now reaches U4.6
- net u4-6: now also U17.1
- net rp2-1: now reaches RP2.1 (R1.1)
- net rp2-2: now reaches RP2.2 (R1.2)
- net rp2-3: now reaches RP2.3 (R2.1)
- net u4-1: now reaches U4.1
- net rp5-6: now reaches RP5.6 (R3.2)
- net rp5-8: now reaches RP5.8 (R4.2)
- net rp3-2: now reaches RP3.2 (R1.2)
- net rp6-1: now reaches RP6.1 (R1.1)
- net rp4-4: now reaches RP4.4 (R2.2)
- net rp8-8: now reaches U10.143
- net rp8-8: now also RP8.8 (R4.2)
- net rp8-5: now reaches U10.144
- net rp8-5: now also RP8.5 (R3.1)
- net u10-153: now reaches U10.153
- net d3-2: no longer names the net of D3.2 (A), JP9.1 (Pin_1)
- net d4-2: no longer names the net of D4.1 (K), R49.1
- net jp1-2 renamed turbo
- net turbo: now also TURBO1.2 (Pin_2)
- net q3-3: no longer names the net of Q3.3 (B), R47.2
- net r46-2: no longer names the net of R45.2, R46.2
- net r46-2: now also Q2.3 (B)
- net r47-1: no longer names the net of R47.1
- net r47-1: now also Q2.2 (C)
- new net key-1: KEYLOCK1.1 (Pin_1)
- new net q1-2: Q1.2 (C)
- new net q1-3: Q1.3 (B), R10.2
- new net spk-1: J17.1 (Pin_1), J17.4 (Pin_4)
- new net spk-2: J17.2 (Pin_2), J17.3 (Pin_3)
- no-connect marks 35 -> 49
Other:
- moved on the sheet: BT1, C58, CON1, CON2, D2, D3, D4, J11, JP9, Q3, R45, R46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

Commit message: PAL decoding
Parts:
- renumbered J17 to J17(HDDLED)1
Connections:
- net con1-10 renamed HDD_D11
- net con1-12 renamed HDD_D12
- net con1-14 renamed HDD_D13
- net con1-16 renamed HDD_D14
- net con1-18 renamed HDD_D15
- net con1-3 renamed HDD_D7
- net con1-39 renamed ~{HDD_ACT}
- net con1-4 renamed HDD_D8
- net con1-5 renamed HDD_D6
- net con1-6 renamed HDD_D9
- net con1-7 renamed HDD_D5
- net con1-8 renamed HDD_D10
- net jp15-1 renamed j12-irq14
- net jp15-2 renamed HDD_INTRQ
- net u1-2 renamed HDD_D0
- net u1-3 renamed HDD_D1
- net u1-4 renamed HDD_D2
- net u1-5 renamed HDD_D3
- net u1-6 renamed HDD_D4
- net u20-18 renamed ~{IDE_CS1}
- net u4-1 renamed ~{IDE_CS0}
Other:
- note added: "(~{1F0-1F7}, ~{3F6-3F7}) if IOR=1"
- note added: "(~{1F0-1F7}, ~{3F6}) if IOR=0"
- note added: "000-00F DMA Controller 010-01F DMA Controller (PS/2) 020-02F Master Programmable Interrupt Controller (PIC) 030-03F Slave PIC 040-05F Programmable Interval Timer (PIT) 060-06F Keyboard Controller 070-071 Real Time Clock 080-083 DMA Page Registers 090-097 Programmable Option Select (PS/2) 0A0-0AF PIC #2 0C0-0CF DMAC #2 0E0-0EF reserved 0F0-0FF Math coprocessor, PCJr Disk Controller 100-10F Program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"
- note added: "1F0-1FF Hard Drive 0 (AT) 3F0-3F7 Floppy Disk Controller"
- note added: "Enable all: AEN = 0"
- note added: "Enable all: JP14 = 1"
- note added: "~{1F0-1F7}"
- note added: "~{1F0-1F7}, ~{3F6-3F7}"
- note added: "~{3F0-3F7}"
- moved on the sheet: U20

Commit message: PCB update
Parts:
- added C34, C49, C53: ~, Capacitor_THT:C_Disc_D4.3mm_W1.9mm_P5.00mm, symbol Device:C_Small
- added C54, C55, C61, C66: 10u, Capacitor_THT:CP_Radial_D5.0mm_P2.50mm, symbol Device:C_Polarized_Small
- added C59, C67: DNP, Capacitor_THT:C_Disc_D3.0mm_W1.6mm_P2.50mm, symbol Device:C_Small
- added R11, R56, R59: R_Small, Resistor_THT:R_Axial_DIN0204_L3.6mm_D1.6mm_P5.08mm_Horizontal, symbol Device:R_Small
- added RAM1, RAM10, RAM2, RAM3, RAM4, RAM7, RAM8, RAM9: M5M44256BP, Package_DIP:CERDIP-20_W7.62mm_SideBrazed, symbol _mine_d:M5M44256
- added U9: 27C512, Package_DIP:DIP-28_W15.24mm, symbol Memory_EPROM:27C512
Connections:
- net +5V: now also RAM1.10 (VCC), RAM10.10 (VCC), RAM2.10 (VCC), RAM3.10 (VCC), RAM4.10 (VCC), RAM7.10 (VCC), RAM8.10 (VCC), RAM9.10 (VCC), U9.28 (VCC)
- net GND: now also RAM1.20 (VSS), RAM10.20 (VSS), RAM2.20 (VSS), RAM3.20 (VSS), RAM4.20 (VSS), RAM7.20 (VSS), RAM8.20 (VSS), RAM9.20 (VSS), U9.14 (GND)
- net u6-89: now also RAM2.2 (DQ2)
- net u6-90: now also RAM10.2 (DQ2)
- net u6-93: now also RAM2.1 (DQ1)
- net u11-6: now reaches U11.6 (A4)
- net u11-6: now also RAM3.19 (DQ4)
- net u11-7: now reaches U11.7 (A5)
- net u11-7: now also RAM3.18 (DQ3)
- net ram3-1: now reaches U11.9 (A7)
- net ram3-1: now also RAM3.1 (DQ1)
- new net ram1-1: RAM1.1 (DQ1)
- new net ram1-12: RAM1.12 (A5)
- new net ram1-18: RAM1.18 (DQ3), RAM7.18 (DQ3), U9.13 (D2)
- new net ram1-19: RAM1.19 (DQ4), RAM7.19 (DQ4), U9.15 (D3)
- new net ram1-2: RAM1.2 (DQ2)
- new net ram1-8: RAM1.8 (A2), RAM10.8 (A2), RAM7.8 (A2), RAM8.8 (A2), RAM9.8 (A2)
- new net ram1-9: RAM1.9 (A3), RAM7.9 (A3)
- new net ram10-13: RAM10.13 (A6)
- new net ram2-12: RAM2.12 (A5), RAM8.12 (A5)
- new net ram2-18: RAM2.18 (DQ3), RAM8.18 (DQ3)
- new net ram2-19: RAM2.19 (DQ4)
- new net ram2-3: RAM2.3 (~{W}), RAM8.3 (~{W})
- new net ram2-7: RAM2.7 (A1), RAM8.7 (A1)
- new net ram3-13: RAM3.13 (A6), RAM9.13 (A6)
- new net ram3-2: RAM3.2 (DQ2), RAM9.2 (DQ2)
- new net ram3-6: RAM3.6 (A0), RAM9.6 (A0)
- new net ram4-1: RAM10.1 (DQ1), RAM4.1 (DQ1)
- new net ram4-11: RAM10.11 (A4), RAM4.11 (A4)
- new net ram4-12: RAM4.12 (A5)
- new net ram4-14: RAM10.14 (A7), RAM4.14 (A7)
- new net ram4-3: RAM10.3 (~{W}), RAM4.3 (~{W})
- new net ram7-6: RAM7.6 (A0)
- new net ram9-15: RAM3.15 (A8), RAM9.15 (A8)

Commit message: PCB update
Connections:
- net bk4-1 is gone; now on net u6-117: BKSW4.1 (Pin_1), RP6.4 (R2.2)
- net ram1-12 is gone; now on net ram4-12: RAM1.12 (A5)
- net ram10-13 is gone; now on net ram3-13: RAM10.13 (A6)
- net ram2-12 is gone; now on net ram4-12: RAM2.12 (A5), RAM8.12 (A5)
- net ram4-11 is gone; now on net ram3-11: RAM10.11 (A4), RAM4.11 (A4)
- net ram7-6 is gone; now on net ram3-6: RAM7.6 (A0)
- net ram9-15 is gone; now on net ram3-15: RAM3.15 (A8), RAM9.15 (A8)
- net rp3-2 is gone; now on net u6-139: RP3.2 (R1.2)
- net rp6-1 is gone; now on net ram1-17: RP6.1 (R1.1)
- net spk-2 is gone; now on net ~{HDD_ACT}: J17(HDDLED)1.2 (Pin_2), J17(HDDLED)1.3 (Pin_3)
- net u6-143 is gone; now on net rp5-6: U6.143
- net u6-77 is gone; now on net ram2-19: U6.77
- net u6-78 is gone; now on net ram4-19: U11.2 (A0), U6.78
- net u6-85 is gone; now on net ram2-18: U6.85
- net u6-86 is gone; now on net ram4-18: U11.3 (A1), U6.86
- net u6-97 is gone; now on net ram1-19: U6.97
- net GND: now also RAM1.16 (~{OE}), RAM10.16 (~{OE}), RAM2.16 (~{OE}), RAM3.16 (~{OE}), RAM4.16 (~{OE}), RAM7.16 (~{OE}), RAM8.16 (~{OE}), RAM9.16 (~{OE})
- net ram1-1: now also RAM7.1 (DQ1)
- net ram1-2: now also RAM7.2 (DQ2)
- net ram1-8: now also RAM2.8 (A2), RAM3.8 (A2), RAM4.8 (A2)
- net ram1-9: now also RAM10.9 (A3), RAM2.9 (A3), RAM3.9 (A3), RAM4.9 (A3), RAM8.9 (A3), RAM9.9 (A3)
- net ram2-19: now also RAM8.19 (DQ4)
- net ram2-3: now also RAM1.3 (~{W}), RAM7.3 (~{W})
- net ram2-7: now also RAM1.7 (A1), RAM10.7 (A1), RAM3.7 (A1), RAM4.7 (A1), RAM7.7 (A1), RAM9.7 (A1)
- net ram3-1: now also RAM9.1 (DQ1)
- net ram3-13: now also RAM1.13 (A6), RAM2.13 (A6), RAM4.13 (A6), RAM7.13 (A6), RAM8.13 (A6)
- net ram3-2: now also U11.8 (A6)
- net ram3-6: now also RAM1.6 (A0), RAM10.6 (A0), RAM2.6 (A0), RAM4.6 (A0), RAM8.6 (A0)
- net ram4-12: now also RAM10.12 (A5), RAM3.12 (A5), RAM7.12 (A5), RAM9.12 (A5)
- net ram4-14: now also RAM1.14 (A7), RAM2.14 (A7), RAM3.14 (A7), RAM7.14 (A7), RAM8.14 (A7), RAM9.14 (A7)
- net ram4-3: now also RAM3.3 (~{W}), RAM9.3 (~{W})
- net rp5-8: now also R62.1, U6.142
- net u11-6: now also RAM9.19 (DQ4)
- net u11-7: now also RAM9.18 (DQ3)
- net u15-5: now also U9.23 (A11)
- net u15-6: now also U9.2 (A12)
- net u19-15: now also U9.26 (A13)
- net u6-115: now also U9.22 (~{OE})
- net u6-124: no longer U6.142
- net u6-138: now also RP3.4 (R2.2)
- net u6-71: now also U9.21 (A10)
- net u6-89: now also RAM8.2 (DQ2)
- net u6-90: now also RAM4.2 (DQ2)
- net u6-93: now also RAM8.1 (DQ1)
- net bk3-2: now reaches BKSW3.2 (Pin_2)
- net ram3-11: now reaches RAM2.11 (A4)
- net ram3-11: now also RAM1.11 (A4), RAM3.11 (A4), RAM7.11 (A4), RAM8.11 (A4), RAM9.11 (A4)
- net ram3-15: now reaches RAM2.15 (A8)
- net ram3-15: now also RAM1.15 (A8), RAM10.15 (A8), RAM4.15 (A8), RAM7.15 (A8), RAM8.15 (A8)
- net ram1-17: now reaches RAM2.17 (~{CAS})
- net ram1-17: now also RAM1.17 (~{CAS}), RAM3.17 (~{CAS}), RAM4.17 (~{CAS})
- net ram1-4: now reaches RAM2.4 (~{RAS})
- net ram1-4: now also RAM1.4 (~{RAS}), RAM3.4 (~{RAS}), RAM4.4 (~{RAS})
- net ram7-17: now reaches RAM10.17 (~{CAS})
- net ram7-17: now also RAM7.17 (~{CAS}), RAM8.17 (~{CAS}), RAM9.17 (~{CAS})
- net ram4-18: now reaches RAM10.18 (DQ3)
- net ram4-18: now also RAM4.18 (DQ3)
- net ram4-19: now reaches RAM10.19 (DQ4)
- net ram4-19: now also RAM4.19 (DQ4)
- net ram7-4: now reaches RAM10.4 (~{RAS})
- net ram7-4: now also RAM7.4 (~{RAS}), RAM8.4 (~{RAS}), RAM9.4 (~{RAS})
- net bk1-2: now reaches BKSW1.2 (Pin_2)
- net bk1-2: now also RP2.5 (R3.1)
- net rp2-4: now reaches RP2.4 (R2.2)
- net rp2-6: now reaches RP2.6 (R3.2)
- net rp2-8: now reaches RP2.8 (R4.2)
- net rp5-1: now reaches RP5.1 (R1.1)
- net rp3-1: now reaches RP3.1 (R1.1)
- net rp4-1: now reaches RP4.1 (R1.1)
- net spk-1 renamed hddled1

Commit message: PCB update
Parts:
- added RAM11, RAM12, RAM5, RAM6: MN41256A, Package_DIP:CERDIP-16_W7.62mm_SideBrazed, symbol _mine_d:MN41256
- Q1, Q2, Q3, Q4: footprint Package_TO_SOT_THT:TO-92_Inline_Wide -> Package_TO_SOT_THT:TO-92_Inline
Connections:
- net ram1-9 is gone; now on net MA3: RAM1.9 (A3), RAM10.9 (A3), RAM2.9 (A3), RAM3.9 (A3), RAM4.9 (A3), RAM7.9 (A3), RAM8.9 (A3), RAM9.9 (A3)
- net ram3-13 is gone; now on net MA6: RAM1.13 (A6), RAM10.13 (A6), RAM2.13 (A6), RAM3.13 (A6), RAM4.13 (A6), RAM7.13 (A6), RAM8.13 (A6), RAM9.13 (A6)
- net ram3-6 is gone; now on net MA0: RAM1.6 (A0), RAM10.6 (A0), RAM2.6 (A0), RAM3.6 (A0), RAM4.6 (A0), RAM7.6 (A0), RAM8.6 (A0), RAM9.6 (A0)
- net ram4-12 is gone; now on net MA5: RAM1.12 (A5), RAM10.12 (A5), RAM2.12 (A5), RAM3.12 (A5), RAM4.12 (A5), RAM7.12 (A5), RAM8.12 (A5), RAM9.12 (A5)
- net rp3-1 is gone; now on net MA4: RP3.1 (R1.1)
- net rp4-1 is gone; now on net MA8: RP4.1 (R1.1)
- net u6-127 is gone; now on net rp2-2: BKSW1.1 (Pin_1), U6.127
- net u6-134 is gone; now on net rp4-4: U6.134
- net u6-136 is gone; now on net rp4-6: U6.136
- net u6-137 is gone; now on net rp4-8: U6.137
- net +5V: now also RAM11.8 (VDD), RAM12.8 (VDD), RAM5.8 (VDD), RAM6.8 (VDD)
- net GND: now also RAM11.16 (VSS), RAM12.16 (VSS), RAM5.16 (VSS), RAM6.16 (VSS)
- net ram1-17: now also RAM5.15 (~{CAS}), RAM6.15 (~{CAS})
- net ram2-3: now also RAM11.3 (~{W}), RAM5.3 (~{W})
- net u6-132: now also RP5.2 (R1.2)
- net u6-133: now also RP5.4 (R2.2)
- net ram6-3: now reaches RP5.3 (R2.1)
- net ram6-3: now also RAM6.3 (~{W})
- net MA0: now reaches RP5.5 (R3.1)
- net MA0: now also RAM11.5 (A0), RAM12.5 (A0), RAM5.5 (A0), RAM6.5 (A0)
- net MA5: now reaches RP3.3 (R2.1)
- net MA5: now also RAM11.10 (A5), RAM12.10 (A5), RAM5.10 (A5), RAM6.10 (A5)
- net MA3: now reaches RP3.5 (R3.1)
- net MA3: now also RAM11.12 (A3), RAM12.12 (A3), RAM5.12 (A3), RAM6.12 (A3)
- net rp6-8: now reaches RP6.8 (R4.2)
- net rp4-3: now reaches RP4.3 (R2.1)
- net rp4-6: now reaches RP4.6 (R3.2)
- net MA6: now reaches RP4.7 (R4.1)
- net MA6: now also RAM11.13 (A6), RAM12.13 (A6), RAM5.13 (A6), RAM6.13 (A6)
- net rp4-8: now reaches RP4.8 (R4.2)
- net ram1-8 renamed MA2
- net MA2: now also RAM11.6 (A2), RAM12.6 (A2), RAM5.6 (A2), RAM6.6 (A2)
- net ram2-7 renamed MA1
- net MA1: now also RAM11.7 (A1), RAM12.7 (A1), RAM5.7 (A1), RAM6.7 (A1)
- net ram3-11 renamed MA4
- net MA4: now also RAM11.11 (A4), RAM12.11 (A4), RAM5.11 (A4), RAM6.11 (A4)
- net ram3-15 renamed MA8
- net MA8: now also RAM11.1 (A8), RAM12.1 (A8), RAM5.1 (A8), RAM6.1 (A8)
- net ram4-14 renamed MA7
- net MA7: now also RAM11.9 (A7), RAM12.9 (A7), RAM5.9 (A7), RAM6.9 (A7)
- net u6-73 renamed ram5-14
- net ram5-14: now also RAM11.14 (Q), RAM11.2 (D), RAM5.14 (Q), RAM5.2 (D)
Other:
- moved on the sheet: C41, RAM1, RAM10, RAM2, RAM3, RAM4, RAM7, RAM8, RAM9, RP1, U1, U11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

Commit message: PCB update
Parts:
- added BANK2_1, BANK2_2, BANK3_1, BANK3_2: SIMM_30_pin, Connector_PinHeader_2.54mm:PinHeader_1x30_P2.54mm_Vertical, symbol _mine_d:SIMM_30_pin
- added JP18, JP6: Conn_01x03, Connector_PinHeader_2.54mm:PinHeader_1x03_P2.54mm_Vertical, symbol Connector_Generic:Conn_01x03
- added RA1, RP12: R_Network08, Resistor_THT:R_Array_SIP9, symbol Device:R_Network08
- Q1, Q2, Q3, Q4: footprint Package_TO_SOT_THT:TO-92_Inline -> Package_TO_SOT_THT:TO-92_Inline_Wide
Connections:
- net ram6-3 is gone; now on net ram4-3: RAM6.3 (~{W}), RP5.3 (R2.1)
- net rp2-1 is gone; now on net ram1-4: RP2.1 (R1.1)
- net rp2-4 is gone; now on net ram7-4: RP2.4 (R2.2)
- net rp5-1 is gone; now on net ram2-3: RP5.1 (R1.1)
- net u6-104 is gone; now on net ram1-18: U6.104
- net u6-105 is gone; now on net u11-7: U6.105
- net u6-108 is gone; now on net ram1-2: U6.108
- net u6-109 is gone; now on net ram3-2: U6.109
- net u6-112 is gone; now on net ram1-1: U6.112
- net u6-113 is gone; now on net ram3-1: U6.113
- net u6-114 is gone; now on net ra1-5: U6.114
- net u6-119 is gone; now on net rp2-3: BKSW2.1 (Pin_1), U6.119
- net u6-74 is gone; now on net ram3-2: U6.74
- net u6-93 is gone; now on net u9-16: RAM2.1 (DQ1), RAM8.1 (DQ1), U6.93
- net u6-94 is gone; now on net ram4-1: U11.5 (A3), U6.94
- net u6-98 is gone; now on net u11-6: U6.98
- net +5V: now also BANK2_1.1 (+5V), BANK2_1.30 (+5V), BANK2_2.1 (+5V), BANK2_2.30 (+5V), BANK3_1.1 (+5V), BANK3_1.30 (+5V), BANK3_2.1 (+5V), BANK3_2.30 (+5V), JP18.1 (Pin_1), RP12.1 (common)
- net GND: now also BANK2_1.22 (GND), BANK2_1.9 (GND), BANK2_2.22 (GND), BANK2_2.9 (GND), BANK3_1.22 (GND), BANK3_1.9 (GND), BANK3_2.22 (GND), BANK3_2.9 (GND), RA1.1 (common)
- net MA0: now also U9.10 (A0), BANK2_1.4 (A0), BANK2_2.4 (A0), BANK3_1.4 (A0), BANK3_2.4 (A0)
- net MA1: now also RP5.7 (R4.1), U9.9 (A1), BANK2_1.5 (A1), BANK2_2.5 (A1), BANK3_1.5 (A1), BANK3_2.5 (A1)
- net MA2: now also RP3.7 (R4.1), U9.8 (A2), BANK2_1.7 (A2), BANK2_2.7 (A2), BANK3_1.7 (A2), BANK3_2.7 (A2)
- net MA3: now also U9.7 (A3), BANK2_1.8 (A3), BANK2_2.8 (A3), BANK3_1.8 (A3), BANK3_2.8 (A3)
- net MA4: now also U9.6 (A4), BANK2_1.11 (A4), BANK2_2.11 (A4), BANK3_1.11 (A4), BANK3_2.11 (A4)
- net MA5: now also U9.5 (A5), BANK2_1.12 (A5), BANK2_2.12 (A5), BANK3_1.12 (A5), BANK3_2.12 (A5)
- net MA6: now also U9.4 (A6), BANK2_1.14 (A6), BANK2_2.14 (A6), BANK3_1.14 (A6), BANK3_2.14 (A6)
- net MA7: now also RP4.5 (R3.1), U9.3 (A7), BANK2_1.15 (A7), BANK2_2.15 (A7), BANK3_1.15 (A7), BANK3_2.15 (A7)
- net MA8: now also U9.25 (A8), BANK2_1.17 (A8), BANK2_2.17 (A8), BANK3_1.17 (A8), BANK3_2.17 (A8)
- net bk3-2: now also RP6.5 (R3.1)
- net ram1-1: now also U9.11 (D0), BANK2_1.3 (D0), BANK3_1.3 (D0)
- net ram1-18: now also BANK2_1.10 (D2), BANK3_1.10 (D2)
- net ram1-19: now also BANK2_1.13 (D3), BANK3_1.13 (D3)
- net ram1-2: now also U9.12 (D1), BANK2_1.6 (D1), BANK3_1.6 (D1)
- net ram1-4: now also RAM5.4 (~{RAS}), RAM6.4 (~{RAS})
- net ram2-18: now also U9.18 (D6), BANK2_1.23 (D6), BANK3_1.23 (D6)
- net ram2-19: now also U9.19 (D7), BANK2_1.25 (D7), BANK3_1.25 (D7)
- net ram2-3: now also BANK2_1.21 (~{WE}), BANK3_1.21 (~{WE})
- net ram3-1: now also BANK2_2.3 (D0), BANK3_2.3 (D0), RP12.4 (R3)
- net ram3-2: now also RAM12.14 (Q), RAM12.2 (D), RAM6.14 (Q), RAM6.2 (D), BANK2_2.26 (QP), BANK2_2.29 (DP), BANK2_2.6 (D1), BANK3_2.26 (QP), BANK3_2.29 (DP), BANK3_2.6 (D1), RP12.3 (R2)
- net ram4-1: now also BANK2_2.16 (D4), BANK3_2.16 (D4), RP12.8 (R7)
- net ram4-18: now also BANK2_2.23 (D6), BANK3_2.23 (D6), RP12.7 (R6)
- net ram4-19: now also BANK2_2.25 (D7), BANK3_2.25 (D7), RP12.9 (R8)
- net ram4-3: now also RAM12.3 (~{W}), BANK2_2.21 (~{WE}), BANK3_2.21 (~{WE})
- net ram5-14: now also BANK2_1.26 (QP), BANK2_1.29 (DP), BANK3_1.26 (QP), BANK3_1.29 (DP)
- net ram7-17: now also RAM11.15 (~{CAS}), RAM12.15 (~{CAS}), RP6.3 (R2.1)
- net ram7-4: now also RAM11.4 (~{RAS}), RAM12.4 (~{RAS})
- net rp2-6: now also BANK2_1.27 (~{RAS}), BANK2_2.27 (~{RAS})
- net rp2-8: now also BANK3_1.27 (~{RAS}), BANK3_2.27 (~{RAS})
- net rp4-3: now also U9.24 (A9), BANK2_1.18 (A9), BANK2_2.18 (A9), BANK3_1.18 (A9), BANK3_2.18 (A9)
- net rp6-8: now also BANK3_1.2 (~{CAS}), BANK3_1.28 (~{CASP}), BANK3_2.2 (~{CAS}), BANK3_2.28 (~{CASP})
- net u11-6: now also BANK2_2.13 (D3), BANK3_2.13 (D3), RP12.5 (R4)
- net u11-7: now also BANK2_2.10 (D2), BANK3_2.10 (D2), RP12.2 (R1)
- net u6-125: now also RP6.2 (R1.2)
- net u6-141: now also RA1.2 (R1)
- net u6-89: now also U9.17 (D5), BANK2_1.20 (D5), BANK3_1.20 (D5)
- net u6-90: now also BANK2_2.20 (D5), BANK3_2.20 (D5), RP12.6 (R5)
- net jp18-2: now reaches U9.1 (A15)
- net jp18-2: now also JP18.2 (Pin_2)
- net u9-16: now reaches U9.16 (D4)
- net u9-16: now also BANK2_1.16 (D4), BANK3_1.16 (D4)
- net ra1-5: now reaches U9.20 (~{CE})
- net ra1-5: now also RA1.5 (R4)
- net jp6-2: now reaches U9.27 (A14)
- net jp6-2: now also JP6.2 (Pin_2)
- net spkr1: now reaches SPEAKER1.1 (Pin_1)
- net rp6-6: now reaches RP6.6 (R3.2)
- net rp6-6: now also BANK2_1.2 (~{CAS}), BANK2_1.28 (~{CASP}), BANK2_2.2 (~{CAS}), BANK2_2.28 (~{CASP})
- net u19-16 renamed jp6-3
- net jp6-3: now also JP6.3 (Pin_3)
- net u19-18 renamed jp18-3
- net jp18-3: now also JP18.3 (Pin_3), JP6.1 (Pin_1)
- no-connect marks 49 -> 57
Other:
- moved on the sheet: C41, RAM1, RAM10, RAM11, RAM12, RAM2, RAM3, RAM4, RAM5, RAM6, RAM7, RAM8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
