File: KiCAD/286.kicad_sch (KiCad schematic)
At the start: 156 parts, among them CON1 Conn_02x20_Odd_Even, CON2 Conn_02x17_Odd_Even, J10 Bus_ISA_16bit, J11 Bus_ISA_16bit, J12 Bus_ISA_16bit, J17(HDDLED)1 Conn_01x04, J9 Bus_ISA_16bit, Q1 2SC1815, Q2 2SC1815, Q3 2SA1015, Q4 2SC1815, U1 74LS245, U10 ST62C303-A, U11 74LS245, U12 74LS00, U14 74LS06, U15 HM6818P, U16 4069, U17 74AHCT125, U18 74LS245, U19 D8041AHC, U20 PAL16L8, U3 74LS245, U4 74LS32, U5 80C287, U6 ST62C241-A, U7 N80L286-16/S, U8 MCS3201FN, U9 27C512, X1 Crystal, X2 Crystal

Commit message: PCB update
Parts:
- removed RP6: 40R, Resistor_THT:R_Array_SIP8, symbol Device:R_Pack04_SIP
- added R12, R16, R60, R9: R_Small, _mine:R_Axial_L3.6mm_D1.6mm_P4.5mm_Horizontal, symbol Device:R_Small
- added unit 3 of RP11
- added unit 2 of RP11
- added unit 4 of RP11
- added RP6: R_Pack04_SIP_Split, Resistor_THT:R_Array_SIP8, symbol Device:R_Pack04_SIP_Split
- added SW1: Conn_02x08_Odd_Even, Connector_PinHeader_2.54mm:PinHeader_2x08_P2.54mm_Vertical, symbol Connector_Generic:Conn_02x08_Odd_Even
- RP11: symbol Device:R_Network04 -> Device:R_Network04_Split
Connections:
- net u6-128 is gone; now on net dl1-in: U6.128
- net u6-35 is gone; now on net u19-8: RP10.3 (R2), U10.131, U6.35
- net +5V: now also RP11.1 (R1), RP11.1 (R1), RP11.1 (R1)
- net bk3-2: now also RP6.5 (R3.1)
- net bk4-2: now also RP6.7 (R4.1)
- net hddled1: now also R16.1
- net key-1: now also R12.1
- net q1-2: now also R11.2
- net ram1-17: now also RP6.1 (R1.1)
- net ram3-2: no longer BANK2_2.26 (QP), BANK2_2.29 (DP), BANK3_2.26 (QP), BANK3_2.29 (DP), RAM12.14 (Q), RAM12.2 (D), RAM6.14 (Q), RAM6.2 (D), U6.74
- net ram7-17: now also RP6.3 (R2.1)
- net rp11-5: now also RP11.5 (R4.2); no longer RP11.5 (R4)
- net rp6-6: now also RP6.6 (R3.2)
- net rp6-8: now also RP6.8 (R4.2)
- net u10-153: now also R56.1
- net u6-117: now also RP6.4 (R2.2)
- net u6-125: now also RP6.2 (R1.2)
- net ~{ERROR}: now also RP11.4 (R3.2); no longer RP11.4 (R3)
- net dl1-in: now reaches DL1.1 (IN)
- net sw1-5: now reaches RA1.3 (R2)
- net sw1-5: now also SW1.5 (Pin_5)
- net sw1-13: now reaches RA1.4 (R3)
- net sw1-13: now also SW1.13 (Pin_13)
- net sw1-7: now reaches RA1.6 (R5)
- net sw1-7: now also SW1.7 (Pin_7)
- net sw1-9: now reaches RA1.7 (R6)
- net sw1-9: now also SW1.9 (Pin_9)
- net sw1-11: now reaches RA1.8 (R7)
- net sw1-11: now also SW1.11 (Pin_11)
- net sw1-15: now reaches RA1.9 (R8)
- net sw1-15: now also SW1.15 (Pin_15)
- net reset_jumper: now reaches RESET1.2 (Pin_2)
- net turbo1: now reaches TUR-LED1.1 (Pin_1)
- net turbo1: now also R9.2
- net pr11-3 renamed sw1-4
- net sw1-4: now also RP11.3 (R2.2), SW1.4 (Pin_4); no longer RP11.3 (R2)
- net rp4-4 renamed sw1-6
- net sw1-6: now also SW1.6 (Pin_6)
- net rp4-6 renamed sw1-10
- net sw1-10: now also SW1.10 (Pin_10)
- net rp4-8 renamed sw1-12
- net sw1-12: now also SW1.12 (Pin_12)
- net u19-33 renamed sw1-2
- net sw1-2: now also SW1.2 (Pin_2)
- net u6-135 renamed sw1-8
- net sw1-8: now also SW1.8 (Pin_8)
- net u6-138 renamed sw1-14
- net sw1-14: now also SW1.14 (Pin_14)
- net u6-139 renamed sw1-16
- net sw1-16: now also SW1.16 (Pin_16)
- new net ram6-2: BANK2_2.26 (QP), BANK2_2.29 (DP), BANK3_2.26 (QP), BANK3_2.29 (DP), RAM12.14 (Q), RAM12.2 (D), RAM6.14 (Q), RAM6.2 (D), U6.74
- new net sw1-3: SW1.3 (Pin_3)
Other:
- moved on the sheet: C46, C47, DL1, JP18, JP6, U10, U14A, U14B, U14C, U14D, U14E, U14F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

Commit message: PCB update
Parts:
- RP6: value R_Pack04_SIP_Split -> 47R
Connections:
- net q4-2 is gone; now on net tur_led: Q4.2 (C)
- net u6-45 is gone; now on net sw1-3: U6.45
- net u6-53 is gone; now on net reset_jumper: C7.1, D1.2 (A), RA7.7 (R6), U14.10, U15.16 (~{STBY}), U6.53
- net +5V: now also R12.2, R16.2, R59.1, R60.1, R9.1
- net j12-io: now also R59.2
- net j12-smemw: now also R56.2
- net spkr1: now also R11.1
- net tur_led: now reaches TUR-LED1.2 (Pin_2)
- net q1-2: no longer names the net of Q1.2 (C), R11.2
- net q1-3: no longer names the net of Q1.3 (B), R10.2
- net r1-1: no longer names the net of Q4.3 (B), R1.1
- net ram1-1 renamed MD0
- net ram1-17 renamed ~{M0_CAS}
- net ram1-18 renamed MD2
- net ram1-19 renamed MD3
- net ram1-2 renamed MD1
- net ram1-4 renamed ~{M0_RAS}
- net ram2-18 renamed MD6
- net ram2-19 renamed MD7
- net ram3-1 renamed MD8
- net ram3-2 renamed MD9
- net ram4-1 renamed MD12
- net ram4-18 renamed MD14
- net ram4-19 renamed MD15
- net ram7-17 renamed ~{M1_CAS}
- net ram7-4 renamed ~{M1_RAS}
- net rp2-6 renamed ~{M2_RAS}
- net rp2-8 renamed ~{M3_RAS}
- net rp6-6 renamed ~{M2_CAS}
- net rp6-8 renamed ~{M3_CAS}
- net u11-6 renamed MD11
- net u11-7 renamed MD10
- net u6-89 renamed MD5
- net u6-90 renamed MD13
- net u9-16 renamed MD4
Other:
- moved on the sheet: BKSW1, BKSW2, BKSW3, BKSW4, C7, C76, C77, Q1, Q4, R1, R10, R11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
