File: KiCAD/286.kicad_sch (KiCad schematic)
At the start: 163 parts, among them CON1 Conn_02x20_Odd_Even, CON2 Conn_02x17_Odd_Even, J10 Bus_ISA_16bit, J11 Bus_ISA_16bit, J12 Bus_ISA_16bit, J17(HDDLED)1 Conn_01x04, J7 Bus_ISA_8bit_narrow, J8 Bus_ISA_8bit_narrow, J9 Bus_ISA_16bit, Q1 2SC1815, Q2 2SC1815, Q3 2SA1015, Q4 2SC1815, SW1 Conn_02x08_Odd_Even, U1 74LS245, U10 ST62C303-A, U11 74LS245, U12 74LS00, U14 74LS06, U15 HM6818P, U16 4069, U17 74AHCT125, U18 74LS245, U19 D8041AHC, U20 PAL16L8, U3 74LS245, U4 74LS32, U5 80C287, U6 ST62C241-A, U7 N80L286-16/S, U8 MCS3201FN, U9 27C512, X1 14.31818MHz, X2 Crystal

Commit message: schematic update
Parts:
- removed RAM1, RAM2, RAM3, RAM4: M5M44256BP, Package_DIP:CERDIP-20_W7.62mm_SideBrazed, symbol _mine_d:M5M44256
- removed RAM5, RAM6: MN41256A, Package_DIP:CERDIP-16_W7.62mm_SideBrazed, symbol _mine_d:MN41256
- RAM10, RAM7, RAM8, RAM9: symbol _mine_d:M5M44256 -> _mine_d:44256
- RAM11, RAM12: symbol _mine_d:MN41256 -> _mine_d:41256
Other:
- added sheet Memory (Memory.kicad_sch)
- note removed: "BANK0"
- moved on the sheet: RAM10, RAM11, RAM12, RAM7, RAM8, RAM9

Commit message: schematic update
Parts:
- removed BANK2_1, BANK2_2, BANK3_1, BANK3_2: SIMM_30_pin, Connector_PinHeader_2.54mm:PinHeader_1x30_P2.54mm_Vertical, symbol _mine_d:SIMM_30_pin
- removed RAM10, RAM7, RAM8, RAM9: M5M44256BP, Package_DIP:CERDIP-20_W7.62mm_SideBrazed, symbol _mine_d:44256
- removed RAM11, RAM12: MN41256A, Package_DIP:CERDIP-16_W7.62mm_SideBrazed, symbol _mine_d:41256
Connections:
- no-connect marks 65 -> 57
Other:
- note added: "FLOPPY"
- note added: "IDE"
- note removed: "BANK1"
- note removed: "BANK2"
- note removed: "BANK3"
- moved on the sheet: C50, CON2, JP10, JP11, JP18, JP5, JP6, KEYLOCK1, OSC2, Q1, Q4, R1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

Commit message: schematics update
Parts:
- removed BKSW1: B, Connector_PinHeader_2.54mm:PinHeader_1x03_P2.54mm_Vertical, symbol _mine_d:Berg_01x03
- removed BKSW2: K, Connector_PinHeader_2.54mm:PinHeader_1x03_P2.54mm_Vertical, symbol _mine_d:Berg_01x03
- removed BKSW3: J, Connector_PinHeader_2.54mm:PinHeader_1x03_P2.54mm_Vertical, symbol _mine_d:Berg_01x03
- removed BKSW4: P, Connector_PinHeader_2.54mm:PinHeader_1x03_P2.54mm_Vertical, symbol _mine_d:Berg_01x03
- removed BT1: Battery_Cell, _mine:286_bat, symbol Device:Battery_Cell
- removed C17, C18, C25, C28, C30, C31, C32, C34, C38, C40, C41, C43, C44, C45, C46, C47, C49, C53, C60, C62, C76, C77, C80: ~, Capacitor_THT:C_Disc_D4.3mm_W1.9mm_P5.00mm, symbol Device:C_Small
- removed C19, C27, C37, C39, C54, C55, C58, C61, C66, C68: 10u, Capacitor_THT:CP_Radial_D5.0mm_P2.50mm, symbol Device:C_Polarized_Small
- removed C50, C82: DNP, Capacitor_THT:C_Disc_D4.3mm_W1.9mm_P5.00mm, symbol Device:C_Small
- removed C59, C63, C67: DNP, Capacitor_THT:C_Disc_D3.0mm_W1.6mm_P2.50mm, symbol Device:C_Small
- removed C7: 10n, Capacitor_THT:C_Disc_D4.3mm_W1.9mm_P5.00mm, symbol Device:C_Small
- removed CON1: Conn_02x20_Odd_Even, Connector_PinHeader_2.54mm:PinHeader_2x20_P2.54mm_Vertical, symbol Connector_Generic:Conn_02x20_Odd_Even
- removed CON2: Conn_02x17_Odd_Even, Connector_PinHeader_2.54mm:PinHeader_2x17_P2.54mm_Vertical, symbol Connector_Generic:Conn_02x17_Odd_Even
- removed D1, D2, D3, D4: D_Small, Diode_THT:D_A-405_P10.16mm_Horizontal, symbol Device:D_Small
- removed DL1: 31A-5500, _mine:31A-5500, symbol _mine_d:31A-5500
- removed J10, J11, J12, J9: Bus_ISA_16bit, _mine:ISA_16bit, symbol _mine_d:Bus_ISA_16bit_narrow
- removed J17(HDDLED)1, JP9, SPEAKER1: Conn_01x04, Connector_PinHeader_2.54mm:PinHeader_1x04_P2.54mm_Vertical, symbol Connector_Generic:Conn_01x04
- removed J7, J8: Bus_ISA_8bit_narrow, _mine:ISA_8bit, symbol _mine_d:Bus_ISA_8bit_narrow
- removed JP1, JP18, JP19, JP20, JP6, JP7: Conn_01x03, Connector_PinHeader_2.54mm:PinHeader_1x03_P2.54mm_Vertical, symbol Connector_Generic:Conn_01x03
- removed JP10, JP11, JP14, JP15, JP2, JP5, RESET1, TUR-LED1, TURBO1: Conn_01x02, Connector_PinSocket_2.54mm:PinSocket_1x02_P2.54mm_Vertical, symbol Connector_Generic:Conn_01x02
- removed KEYBOARD1: DIN-5, _mine:286_DIN5, symbol Connector:DIN-5
- removed KEYLOCK1: Conn_01x05, Connector_PinHeader_2.54mm:PinHeader_1x05_P2.54mm_Vertical, symbol Connector_Generic:Conn_01x05
- removed OSC1: 32MHz, Oscillator:Oscillator_DIP-14, symbol Oscillator:OCXO-14
- removed OSC2: 24MHz, Oscillator:Oscillator_DIP-14, symbol Oscillator:OCXO-14
- removed OSC3: DNP, Oscillator:Oscillator_DIP-14, symbol Oscillator:OCXO-14
- removed POWER1: Conn_01x12_Pin, Connector_Molex:Molex_KK-396_A-41791-0012_1x12_P3.96mm_Vertical, symbol Connector:Conn_01x12_Pin
- removed Q1, Q2, Q4: 2SC1815, Package_TO_SOT_THT:TO-92L_Inline_Wide, symbol Transistor_BJT:2SC1815
- removed Q3: 2SA1015, Package_TO_SOT_THT:TO-92L_Inline_Wide, symbol Transistor_BJT:2SA1015
- removed R1, R10, R11, R17, R18, R45, R46, R47, R49, R55, R56, R59, R61, R62: R_Small, Resistor_THT:R_Axial_DIN0204_L3.6mm_D1.6mm_P5.08mm_Horizontal, symbol Device:R_Small
- removed R12, R16, R44, R48, R57, R9: R_Small, _mine:R_Axial_L3.6mm_D1.6mm_P4.5mm_Horizontal, symbol Device:R_Small
- removed R14, R53: 30R, Resistor_THT:R_Axial_DIN0204_L3.6mm_D1.6mm_P5.08mm_Horizontal, symbol Device:R_Small
- removed R2: 29R, Resistor_THT:R_Axial_DIN0204_L3.6mm_D1.6mm_P5.08mm_Horizontal, symbol Device:R_Small
- removed R52: 330R, _mine:R_Axial_L3.6mm_D1.6mm_P4.5mm_Horizontal, symbol Device:R_Small
- removed R60: 1k, _mine:R_Axial_L3.6mm_D1.6mm_P4.5mm_Horizontal, symbol Device:R_Small
- removed RA1, RA2, RA3, RA7, RP12: R_Network08, Resistor_THT:R_Array_SIP9, symbol Device:R_Network08
- removed RA5, RA6, RP10: R_Network04, Resistor_THT:R_Array_SIP5, symbol Device:R_Network04
- removed RP1: R_Network09, Resistor_THT:R_Array_SIP10, symbol Device:R_Network09
- removed RP11: R_Network04, Resistor_THT:R_Array_SIP5, symbol Device:R_Network04_Split
- removed RP2, RP3, RP4, RP5: 10R, Resistor_THT:R_Array_SIP8, symbol Device:R_Pack04_SIP_Split
- removed RP6: 47R, Resistor_THT:R_Array_SIP8, symbol Device:R_Pack04_SIP_Split
- removed RP8: R_Pack04_SIP, Resistor_THT:R_Array_SIP8, symbol Device:R_Pack04_SIP
- removed SW1: Conn_02x08_Odd_Even, Connector_PinHeader_2.54mm:PinHeader_2x08_P2.54mm_Vertical, symbol Connector_Generic:Conn_02x08_Odd_Even
- removed U1, U11, U18, U3: 74LS245, Package_DIP:DIP-20_W7.62mm, symbol 74xx:74LS245
- removed U10: ST62C303-A, Package_QFP:PQFP-160_28x28mm_P0.65mm, symbol _mine_d:ST62C303-A
- removed U12: 74LS00, Package_DIP:DIP-14_W7.62mm, symbol 74xx:74LS00
- removed U14: 74LS06, Package_DIP:DIP-14_W7.62mm, symbol 74xx:74LS06
- removed U15: HM6818P, Package_DIP:DIP-24_W15.24mm_Socket, symbol _mine_d:HM6818
- removed U16: 4069, Package_DIP:DIP-14_W7.62mm, symbol 4xxx:4069
- removed U17: 74AHCT125, Package_DIP:DIP-14_W7.62mm, symbol 74xx:74AHCT125
- removed U19: D8041AHC, _mine:DIP-40_W15.24mm_Socket_small_pad, symbol _mine_d:D8041AHC
- removed U20: PAL16L8, Package_DIP:DIP-20_W7.62mm, symbol Logic_Programmable:PAL16L8
- removed U4: 74LS32, Package_DIP:DIP-14_W7.62mm, symbol 74xx:74LS32
- removed U5: 80C287, _mine:DIP-40_W15.24mm_Socket_small_pad, symbol _mine_d:80287
- removed U6: ST62C241-A, Package_QFP:PQFP-160_28x28mm_P0.65mm, symbol _mine_d:ST62C241-A_1
- removed U7: N80L286-16/S, _mine:PLCC-68_from_1, symbol _mine_d:N80L286
- removed U8: MCS3201FN, Package_LCC:PLCC-68, symbol _mine_d:MCS2301
- removed U9: 27C512, Package_DIP:DIP-28_W15.24mm, symbol Memory_EPROM:27C512
- removed X1: 14.31818MHz, Crystal:Crystal_HC50_Horizontal, symbol Device:Crystal
- removed X2: Crystal, Crystal:Crystal_AT310_D3.0mm_L10.0mm_Horizontal, symbol Device:Crystal
Connections:
- no-connect marks 57 -> 0
Other:
- added sheet CPU_ChipSet1 (CPU_ChipSet1.kicad_sch)
- added sheet ChipSet2 (ChipSet2.kicad_sch)
- added sheet FLOPPY_IDE (FLOPPY_IDE.kicad_sch)
- added sheet ISA (ISA.kicad_sch)
- note added: "1MB SIMM30"
- note added: "256kB"
- note added: "80286"
- note added: "80287"
- note added: "A[0..23]"
- note added: "BANK0"
- note added: "BANK1"
- note added: "BANK2"
- note added: "BANK3"
- note added: "CHSET1"
- note added: "CPU"
- note added: "CTRL"
- note added: "D[0..15]"
- note added: "MA[0..9]"
- note added: "MD[0..15], MDP"
- note added: "NPU"
- note added: "PG. 2"
- note added: "PG. 4"
- note added: "ST62C241-A"
- note removed: "(~{1F0-1F7}, ~{3F6-3F7}) if IOR=1"
- note removed: "(~{1F0-1F7}, ~{3F6}) if IOR=0"
- note removed: "000-00F DMA Controller 010-01F DMA Controller (PS/2) 020-02F Master Programmable Interrupt Controller (PIC) 030-03F Slave PIC 040-05F Programmable Interval Timer (PIT) 060-06F Keyboard Controller 070-071 Real Time Clock 080-083 DMA Page Registers 090-097 Programmable Option Select (PS/2) 0A0-0AF PIC #2 0C0-0CF DMAC #2 0E0-0EF reserved 0F0-0FF Math coprocessor, PCJr Disk Controller 100-10F Program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"
- note removed: "1F0-1FF Hard Drive 0 (AT) 3F0-3F7 Floppy Disk Controller"
- note removed: "27256 1-2 27512 2-3"
- note removed: "Bank JP21 JP22 JP23 JP24 SIP RAM as banks 2 & 3 pins 2 & 3 pins 2 & 3 pins 2 & 3 pins 2 & 3 SIP RAM as banks 0 & 1 pins 1 & 2 pins 1 & 2 pins 1 & 2 pins 1 & 2"
- note removed: "Enable all: AEN = 0"
- note removed: "Enable all: JP14 = 1"
- note removed: "FLOPPY"
- note removed: "FLOPPY ENABLE"
- note removed: "Floppy drive address select: 3F4-3F5h Closed 374-375h Open"
- note removed: "Floppy drive speed select: 12MHz Closed 16/20MHz Open"
- note removed: "IDE"
- note removed: "IDE INTERFACE CONFIGURATION Setting JP14 JP15 Enabled Open Closed Disabled Closed Open"
- note removed: "Monitor type select color SW1/1 On Monitor type select monochrome SW1/1 Off Parity enabled SW1/2 On Parity disabled SW1/2 Off"
- note removed: "NPU speed select low (12MHz CPU) JP19 & JP20 pins 1 & 2 closed NPU speed select high (16/20MHz CPU) JP19 & JP20 pins 2 & 3 closed"
- note removed: "~{1F0-1F7}"
- note removed: "~{1F0-1F7}, ~{3F6-3F7}"
- note removed: "~{3F0-3F7}"
- title: (none) -> PC/AT 286
