File: KiCAD/FLOPPY_IDE.kicad_sch (KiCad schematic)
At the start: 20 parts, among them CON1 Conn_02x20_Odd_Even, CON2 Conn_02x17_Odd_Even, J17(HDDLED)1 Conn_01x04, U1 74LS245, U16 4069, U17 74AHCT125, U20 PAL16L8, U3 74LS245, U4 74LS32, U8 MCS3201FN

Commit message: commit from lucky
Parts:
- JP11, JP5: value Conn_01x02 -> DNP
Other:
- moved on the sheet: C50, CON1, CON2, J17(HDDLED)1, JP10, JP11, JP14, JP15, JP5, OSC2, R16, R2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
