File: KiCAD/CPU_ChipSet1.kicad_sch (KiCad schematic)
At the start: 87 parts, among them Q4 2SC1815, SW1 Conn_02x08_Odd_Even, U12 74LS00, U14 74LS06, U16 4069, U17 74AHCT125, U19 D8041AHC, U4 74LS32, U5 80C287, U6 ST62C241-A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

Commit message: IDE controller update
Other:
- note added: "(14.3MHz)"
- note added: "(7.14MHz)"
Changed lines of the file:
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@@
 		)
 	)
+	(text "(7.14MHz)"
+		(exclude_from_sim no)
+		(at 263.652 199.644 0)
+		(effects
+			(font
+				(size 1.27 1.27)
+			)
+		)
+	)
 	(text "NPU speed select low (12MHz CPU) JP19 & JP20 pins 1 & 2 closed\nNPU speed select high (16/20MHz CPU) JP19 & JP20 pins 2 & 3 closed"
 		(exclude_from_sim no)
@@
 		)
 	)
+	(text "(14.3MHz)"
+		(exclude_from_sim no)
+		(at 163.576 200.914 0)
+		(effects
+			(font
+				(size 1.27 1.27)
+			)
+		)
+	)
 	(text "Monitor type select color SW1/1 On\nMonitor type select monochrome SW1/1 Off\nParity enabled SW1/2 On\nParity disabled SW1/2 Off"
 		(exclude_from_sim no)
@@
 		)
 	)
+	(text "(7.14MHz)"
+		(exclude_from_sim no)
+		(at 160.274 183.388 0)
+		(effects
+			(font
+				(size 1.27 1.27)
+			)
+		)
+	)
 	(junction
 		(at 29.21 166.37)
@@
 	)
 	(global_label "KBINT"
-		(shape input)
+		(shape output)
 		(at 421.64 383.54 0)
 		(fields_autoplaced yes)

Commit message: 286 sch updates
Connections:
- net D15: now also U7.3 (NC), U7.56 (NC)
- net Net-(JP19-Pin_2): now reaches JP19.2 (Pin_2), U5.39 (CKM)
Other:
- moved on the sheet: C17, JP19, JP20, U5
