File: KiCAD/ChipSet2.kicad_sch (KiCad schematic)
At the start: 39 parts, among them Q1 2SC1815, Q2 2SC1815, Q3 2SA1015, U10 ST62C303-A, U11 74LS245, U12 74LS00, U15 HM6818P, U16 4069, U18 74LS245, X1 14.31818MHz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

Commit message: 286 sch updates
Parts:
- X2: value Crystal -> 32.768kHz
Changed lines of the file:
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@@
 	(wire
 		(pts
+			(xy 331.47 109.22) (xy 323.85 109.22)
+		)
+		(stroke
+			(width 0)
+			(type default)
+		)
+	)
+	(wire
+		(pts
 			(xy 157.48 139.7) (xy 179.07 139.7)
 		)
@@
 		)
 	)
-	(label "~{RTCCE}"
-		(at 323.85 109.22 0)
-		(effects
-			(font
-				(size 1.27 1.27)
-			)
-			(justify left bottom)
-		)
-	)
 	(label "+5V"
 		(at 101.6 27.94 90)
@@
 		)
 	)
+	(global_label "~{RTCCE}"
+		(shape input)
+		(at 331.47 109.22 0)
+		(fields_autoplaced yes)
+		(effects
+			(font
+				(size 1.27 1.27)
+			)
+			(justify left)
+		)
+		(property "Intersheetrefs" "${INTERSHEET_REFS}"
+			(at 340.3818 109.22 0)
+			(effects
+				(font
+					(size 1.27 1.27)
+				)
+				(justify left)
+			)
+		)
+	)
 	(global_label "CHSET03"
 		(shape bidirectional)
@@
 			)
 		)
-		(property "Value" "Crystal"
+		(property "Value" "32.768kHz"
 			(at 243.84 78.74 0)
 			(effects
