File: IDE_controller/IDE_controller/IDE_controller.kicad_pcb (KiCad board)
At the start: 2 copper layers, 14 parts, among them J1 Bus_ISA_16bit_narrow, J10 Conn_01x02, U12 74LS245, U13 74LS245

Commit message: IDE controller update
Parts:
- added CON2: Conn_02x17_Odd_Even, Connector_PinHeader_2.54mm:PinHeader_2x17_P2.54mm_Vertical, F.Cu at (82.5, 52.6)
- added JP7: Conn_01x03, Connector_PinHeader_2.54mm:PinHeader_1x03_P2.54mm_Vertical, F.Cu at (118.7, 92.7)
- added JP8-1: Conn_01x03, Connector_PinHeader_2.54mm:PinHeader_1x03_P2.54mm_Vertical, F.Cu at (96.8, 92.6)
- added JP8-2: Conn_01x03, Connector_PinHeader_2.54mm:PinHeader_1x03_P2.54mm_Vertical, F.Cu at (99.5, 92.7)
- added JP8-3: Conn_01x03, Connector_PinHeader_2.54mm:PinHeader_1x03_P2.54mm_Vertical, F.Cu at (102.1, 92.7)
- added JP8-4: Conn_01x03, Connector_PinHeader_2.54mm:PinHeader_1x03_P2.54mm_Vertical, F.Cu at (104.5, 92.7)
- added JP8-5: Conn_01x03, Connector_PinHeader_2.54mm:PinHeader_1x03_P2.54mm_Vertical, F.Cu at (107.1, 92.7)
- added JP8-6: Conn_01x03, Connector_PinHeader_2.54mm:PinHeader_1x03_P2.54mm_Vertical, F.Cu at (109.7, 92.6)
- added JP8-7: Conn_01x03, Connector_PinHeader_2.54mm:PinHeader_1x03_P2.54mm_Vertical, F.Cu at (112.3, 92.7)
- added JP8-8: Conn_01x03, Connector_PinHeader_2.54mm:PinHeader_1x03_P2.54mm_Vertical, F.Cu at (114.9, 92.6)
- added U11: C820101A, _mine:LQFP-48_10x10mm_P0.7mm, F.Cu at (141.5, 104.1)
Connections:
- J1 pad 1: unconnected-(J1-GND-Pad1) -> /GND
- J1 pad 2: unconnected-(J1-RESET-Pad2) -> RESET
- J1 pad 3: unconnected-(J1-+5V-Pad3) -> /+5V
- J1 pad 4: unconnected-(J1-IRQ2-Pad4) -> IRQ2
- J1 pad 41: unconnected-(J1-IO_READY-Pad41) -> /IO_READY
- J1 pad 42: unconnected-(J1-AEN-Pad42) -> /AEN
- J1 pad 53: unconnected-(J1-BA09-Pad53) -> /BA9
- J1 pad 54: unconnected-(J1-BA08-Pad54) -> /BA8
- J1 pad 55: unconnected-(J1-BA07-Pad55) -> /BA7
- J1 pad 56: unconnected-(J1-BA06-Pad56) -> /BA6
- J1 pad 57: unconnected-(J1-BA05-Pad57) -> /BA5
- J1 pad 58: unconnected-(J1-BA04-Pad58) -> /BA4
- J1 pad 59: unconnected-(J1-BA03-Pad59) -> /BA3
- J1 pad 6: unconnected-(J1-DRQ2-Pad6) -> DRQ2
- J1 pad 60: unconnected-(J1-BA02-Pad60) -> /BA2
- J1 pad 7: unconnected-(J1--12V-Pad7) -> -12V
- J10 pad 2: /j10-2 -> /IO_READY
- R10 pad 2: unconnected-(R10-Pad2) -> /r10-2
- R11 pad 1: unconnected-(R11-Pad1) -> /r11-1
- R11 pad 2: unconnected-(R11-Pad2) -> /r11-2
- R12 pad 2: unconnected-(R12-Pad2) -> /r12-2
- R13 pad 2: unconnected-(R13-Pad2) -> /r13-2
- R14 pad 1: unconnected-(R14-Pad1) -> /u12-19
- R14 pad 2: unconnected-(R14-Pad2) -> /r14-2
- R15 pad 2: unconnected-(R15-Pad2) -> /r15-2
- R7 pad 1: unconnected-(R7-Pad1) -> /r7-1
- R8 pad 2: unconnected-(R8-Pad2) -> /r8-2
- R9 pad 2: unconnected-(R9-Pad2) -> /r9-2
- U12 pad 11: unconnected-(U12-B7-Pad11) -> /HDD_D8
- U12 pad 12: unconnected-(U12-B6-Pad12) -> /HDD_D9
- U12 pad 13: unconnected-(U12-B5-Pad13) -> /HDD_D10
- U12 pad 14: unconnected-(U12-B4-Pad14) -> /HDD_D11
- U12 pad 15: unconnected-(U12-B3-Pad15) -> /HDD_D12
- U13 pad 1: unconnected-(U13-A->B-Pad1) -> /+5V
- U13 pad 10: unconnected-(U13-GND-Pad10) -> /GND
- U13 pad 19: unconnected-(U13-CE-Pad19) -> /GND
- U13 pad 3: /u13-3 -> /BA2
- U13 pad 8: /u13-8 -> /ALE
Routing:
- net /IO_READY: track 0.00 -> 163.1 mm, vias 0 -> 3
- net /BA2: track 0.00 -> 126.0 mm, vias 0 -> 4
- net /j10-2: track 113.8 -> 0.00 mm, vias 3 -> 0
- net /AEN: track 0.00 -> 97.6 mm, vias 0 -> 2
- net /BA1: track 52.4 -> 138.0 mm, vias 2 -> 6
- net /BA0: track 48.3 -> 129.4 mm, vias 1 -> 4
- net /BA9: track 0.00 -> 74.0 mm, vias 0 -> 2
- net /BA3: track 0.00 -> 73.2 mm, vias 0 -> 2
- net /BA4: track 0.00 -> 71.4 mm, vias 0 -> 2
- net /r14-2: track 0.00 -> 70.4 mm, vias 0 -> 1
- net /BA8: track 0.00 -> 69.8 mm, vias 0 -> 2
- net /BA5: track 0.00 -> 69.3 mm, vias 0 -> 2
- net /BA6: track 0.00 -> 67.5 mm, vias 0 -> 2
- net /BA7: track 0.00 -> 67.4 mm, vias 0 -> 2
- net /u13-7: track 0.00 -> 52.7 mm, vias 0 -> 2
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
Commit message: IDE controller update
Parts:
- added JP8: Conn_01x03, Connector_PinHeader_2.54mm:PinHeader_1x03_P2.54mm_Vertical, F.Cu at (157.4, 119.8)
- added JP9-2: Conn_01x03, Connector_PinHeader_2.54mm:PinHeader_1x03_P2.54mm_Vertical, F.Cu at (168.9, 119.8)
- added JP9-3: Conn_01x03, Connector_PinHeader_2.54mm:PinHeader_1x03_P2.54mm_Vertical, F.Cu at (166.4, 119.8)
- added JP9-4: Conn_01x03, Connector_PinHeader_2.54mm:PinHeader_1x03_P2.54mm_Vertical, F.Cu at (163.8, 119.8)
- added JP9-5: Conn_01x03, Connector_PinHeader_2.54mm:PinHeader_1x03_P2.54mm_Vertical, F.Cu at (161.3, 119.8)
- added U14: 74LS245, Package_DIP:DIP-20_W7.62mm, F.Cu at (187.2, 124.9)
- added U2: 74LS125, Package_DIP:DIP-14_W7.62mm, F.Cu at (200.2, 57.5)
- added U4: W86C450, Package_DIP:DIP-40_W15.24mm, F.Cu at (173.2, 64.2)
- added U5: W86C450, Package_DIP:DIP-40_W15.24mm, F.Cu at (154.1, 64.3)
Connections:
- net -12V renamed /-12V
- net /BALE renamed /ALE_IDE
- net DRQ2 renamed /DRQ2
- J1 pad 10: unconnected-(J1-GND-Pad10) -> /GND
- J1 pad 13: unconnected-(J1-~{IOW}-Pad13) -> /~{IOW}
- J1 pad 14: unconnected-(J1-~{IOR}-Pad14) -> /~{IOR}
- J1 pad 2: RESET -> /RESET
- J1 pad 21: unconnected-(J1-IRQ7-Pad21) -> /IRQ7
- J1 pad 22: unconnected-(J1-IRQ6-Pad22) -> /IRQ6
- J1 pad 23: unconnected-(J1-IRQ5-Pad23) -> /IRQ5
- J1 pad 24: unconnected-(J1-IRQ4-Pad24) -> /IRQ4
- J1 pad 25: unconnected-(J1-IRQ3-Pad25) -> /IRQ3
- J1 pad 26: unconnected-(J1-~{DACK2}-Pad26) -> /~{DACK2}
- J1 pad 27: unconnected-(J1-TC-Pad27) -> /TC
- J1 pad 29: unconnected-(J1-VCC-Pad29) -> /+5V
- J1 pad 31: unconnected-(J1-GND-Pad31) -> /GND
- J1 pad 33: unconnected-(J1-DB7-Pad33) -> /DB7
- J1 pad 34: unconnected-(J1-DB6-Pad34) -> /DB6
- J1 pad 35: unconnected-(J1-DB5-Pad35) -> /DB5
- J1 pad 36: unconnected-(J1-DB4-Pad36) -> /DB4
- J1 pad 37: unconnected-(J1-DB3-Pad37) -> /DB3
- J1 pad 38: unconnected-(J1-DB2-Pad38) -> /DB2
- J1 pad 39: unconnected-(J1-DB1-Pad39) -> /DB1
- J1 pad 4: IRQ2 -> /IRQ2
- J1 pad 40: unconnected-(J1-DB0-Pad40) -> /DB0
- J1 pad 91: /D8 -> /DB8
- J1 pad 92: /D9 -> /DB9
- J1 pad 93: /D10 -> /DB10
- J1 pad 94: /D11 -> /DB11
- J1 pad 95: /D12 -> /DB12
- J1 pad 96: /D13 -> /DB13
- J1 pad 97: /D14 -> /DB14
- J1 pad 98: /D15 -> /DB15
- JP5 pad 10: /HDD_D11 -> /D11
- JP5 pad 11: /HDD_D3 -> /D3
- JP5 pad 12: /HDD_D12 -> /D12
- JP5 pad 13: /HDD_D2 -> /D2
- JP5 pad 14: /HDD_D13 -> /D13
- JP5 pad 15: /HDD_D1 -> /D1
- JP5 pad 16: /HDD_D14 -> /D14
- JP5 pad 17: /HDD_D0 -> /D0
- JP5 pad 18: /HDD_D15 -> /D15
- JP5 pad 23: /~{IOW} -> /~{IOW_IDE}
- JP5 pad 25: /~{IOR} -> /~{IOR_IDE}
- JP5 pad 3: /HDD_D7 -> /D7
- JP5 pad 4: /HDD_D8 -> /D8
- JP5 pad 5: /HDD_D6 -> /D6
- JP5 pad 6: /HDD_D9 -> /D9
- JP5 pad 7: /HDD_D5 -> /D5
- JP5 pad 8: /HDD_D10 -> /D10
- JP5 pad 9: /HDD_D4 -> /D4
- U12 pad 1: /~{IOR} -> /~{IOR_IDE}
- U12 pad 11: /HDD_D8 -> /D8
- U12 pad 12: /HDD_D9 -> /D9
- U12 pad 13: /HDD_D10 -> /D10
- U12 pad 14: /HDD_D11 -> /D11
- U12 pad 15: /HDD_D12 -> /D12
- U12 pad 16: /HDD_D13 -> /D13
- U12 pad 17: /HDD_D14 -> /D14
- U12 pad 18: /HDD_D15 -> /D15
- U12 pad 2: /D15 -> /DB15
- U12 pad 3: /D14 -> /DB14
- U12 pad 4: /D13 -> /DB13
- U12 pad 5: /D12 -> /DB12
- U12 pad 6: /D11 -> /DB11
- U12 pad 7: /D10 -> /DB10
- U12 pad 8: /D9 -> /DB9
- U12 pad 9: /D8 -> /DB8
- U13 pad 13: /~{IOR} -> /~{IOR_IDE}
- U13 pad 14: /~{IOW} -> /~{IOW_IDE}
Routing:
- net /D0: track 0.00 -> 186.1 mm, vias 0 -> 2
- net /RESET: track 0.00 -> 115.6 mm, vias 0 -> 2
- net /~{IOR_IDE}: track 0.00 -> 105.4 mm, vias 0 -> 2
- net /~{IOW_IDE}: track 0.00 -> 84.7 mm, vias 0 -> 2
- net /~{IOW}: track 84.7 -> 8.96 mm, vias 2 -> 1
- net /~{IOR}: track 105.4 -> 34.7 mm, vias 2 -> 0
- net /DRQ2: track 0.00 -> 52.0 mm, vias 0 -> 3
- net /HDD_D7: track 51.8 -> 0.00 mm, vias 1 -> 0
- net /D7: track 0.00 -> 51.8 mm, vias 0 -> 1
- net /HDD_D15: track 48.0 -> 0.00 mm, vias 1 -> 0
- net /IRQ2: track 0.00 -> 42.9 mm
- net /HDD_D6: track 42.8 -> 0.00 mm, vias 1 -> 0
- net /D6: track 0.00 -> 42.8 mm, vias 0 -> 1
- net unconnected-(JP9-2-Pin_1-Pad1): track 0.00 -> 41.8 mm, vias 0 -> 1
- net /HDD_D5: track 41.5 -> 0.00 mm, vias 1 -> 0
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