File: IDE_controller/IDE_controller/IDE_controller.kicad_pcb (KiCad board)
At the start: 2 copper layers, 34 parts, among them CON2 Conn_02x17_Odd_Even, J1 Bus_ISA_16bit_narrow, J10 Conn_01x02, U11 C820101A, U12 74LS245, U13 74LS245, U14 74LS245, U2 74LS125, U4 W86C450, U5 W86C450

Commit message: IDE controller update + decoder
Parts:
- added C1: 100n, Capacitor_THT:C_Disc_D4.3mm_W1.9mm_P5.00mm, F.Cu at (131.5, 55.3)
- added C10: 100n, Capacitor_THT:C_Disc_D4.3mm_W1.9mm_P5.00mm, F.Cu at (125.2, 62.9)
- added C11: 100n, Capacitor_THT:C_Disc_D4.3mm_W1.9mm_P5.00mm, F.Cu at (122.9, 108.0)
- added C12: 100n, Capacitor_THT:C_Disc_D4.3mm_W1.9mm_P5.00mm, F.Cu at (78.5, 122.6)
- added C13: 100n, Capacitor_THT:C_Disc_D4.3mm_W1.9mm_P5.00mm, F.Cu at (110.6, 122.8)
- added C14: 100n, Capacitor_THT:C_Disc_D4.3mm_W1.9mm_P5.00mm, F.Cu at (183.9, 122.4)
- added C15: 47p, Capacitor_THT:C_Disc_D4.3mm_W1.9mm_P5.00mm, F.Cu at (213.3, 81.1)
- added C16: 47p, Capacitor_THT:C_Disc_D4.3mm_W1.9mm_P5.00mm, F.Cu at (213.3, 83.8)
- added C17: 10n, Capacitor_THT:C_Disc_D4.3mm_W1.9mm_P5.00mm, F.Cu at (143.5, 80.6)
- added C18: 470p, Capacitor_THT:C_Disc_D4.3mm_W1.9mm_P5.00mm, F.Cu at (146.2, 80.6)
- added C19: 10n, Capacitor_THT:C_Disc_D4.3mm_W1.9mm_P5.00mm, F.Cu at (141.1, 80.6)
- added C2: 100n, Capacitor_THT:C_Disc_D4.3mm_W1.9mm_P5.00mm, F.Cu at (196.9, 55.3)
- added C3: 100n, Capacitor_THT:C_Disc_D4.3mm_W1.9mm_P5.00mm, F.Cu at (201.3, 61.2)
- added C4: 100n, Capacitor_THT:C_Disc_D4.3mm_W1.9mm_P5.00mm, F.Cu at (183.2, 60.9)
- added C5: 100n, Capacitor_THT:C_Disc_D4.3mm_W1.9mm_P5.00mm, F.Cu at (164.0, 61.2)
- added C6: 100n, Capacitor_THT:C_Disc_D4.3mm_W1.9mm_P5.00mm, F.Cu at (175.8, 116.0)
- added C8: 100n, Capacitor_THT:C_Disc_D4.3mm_W1.9mm_P5.00mm, F.Cu at (156.8, 115.9)
- added D1: D_Small, Diode_THT:D_A-405_P10.16mm_Horizontal, F.Cu at (133.4, 75.6)
- added J2: DA15_Socket, Connector_Dsub:DSUB-15_Socket_Horizontal_P2.77x2.54mm_EdgePinOffset9.40mm, F.Cu at (222.4, 55.2)
- added JP1: Conn_01x02, Connector_PinHeader_2.54mm:PinHeader_1x02_P2.54mm_Vertical, F.Cu at (77.0, 57.7)
- added R1: 2k2, Resistor_THT:R_Axial_DIN0207_L6.3mm_D2.5mm_P10.16mm_Horizontal, F.Cu at (209.0, 61.6)
- added R16: 4k6, Resistor_THT:R_Axial_DIN0207_L6.3mm_D2.5mm_P10.16mm_Horizontal, F.Cu at (208.9, 66.5)
- added R17: 4k6, Resistor_THT:R_Axial_DIN0207_L6.3mm_D2.5mm_P10.16mm_Horizontal, F.Cu at (208.9, 64.0)
- added R18: 100R, Resistor_THT:R_Axial_DIN0207_L6.3mm_D2.5mm_P10.16mm_Horizontal, F.Cu at (138.5, 85.7)
- added R19: 2k2, Resistor_THT:R_Axial_DIN0207_L6.3mm_D2.5mm_P10.16mm_Horizontal, F.Cu at (209.0, 74.0)
- added R2: 4k6, Resistor_THT:R_Axial_DIN0207_L6.3mm_D2.5mm_P10.16mm_Horizontal, F.Cu at (209.1, 69.0)
- added R20: 4k6, Resistor_THT:R_Axial_DIN0207_L6.3mm_D2.5mm_P10.16mm_Horizontal, F.Cu at (97.3, 55.9)
- added R3: 4k6, Resistor_THT:R_Axial_DIN0207_L6.3mm_D2.5mm_P10.16mm_Horizontal, F.Cu at (131.0, 85.8)
- added R4: 100R, Resistor_THT:R_Axial_DIN0207_L6.3mm_D2.5mm_P10.16mm_Horizontal, F.Cu at (136.0, 85.8)
- added R5: 4k6, Resistor_THT:R_Axial_DIN0207_L6.3mm_D2.5mm_P10.16mm_Horizontal, F.Cu at (209.0, 71.6)
- added R6: 2k2, Resistor_THT:R_Axial_DIN0207_L6.3mm_D2.5mm_P10.16mm_Horizontal, F.Cu at (209.0, 76.7)
- added U8: UM82C11, Package_DIP:DIP-40_W15.24mm, F.Cu at (191.4, 64.0)
- R10: value 4k6 -> 2k2
- moved JP7 5.08 mm to (118.7, 97.8), turned to 180 degrees
- renumbered JP8-1 to JP6-1, JP8-2 to JP6-2, JP8-3 to JP6-3, JP8-4 to JP6-4, JP8-5 to JP6-5, JP8-6 to JP6-6, JP8-7 to JP6-7, JP8-8 to JP6-8
Connections:
- net /r10-2 renamed Net-(JP6-4-Pin_2)
- net /r11-1 renamed /U8_CS
- net /r11-2 renamed Net-(JP6-5-Pin_2)
- net /r12-2 renamed Net-(JP6-6-Pin_2)
- net /r13-2 renamed Net-(JP6-7-Pin_2)
- net /r14-2 renamed Net-(JP6-8-Pin_2)
- net /r15-2 renamed Net-(JP7-Pin_2)
- net /r7-1 renamed Net-(JP6-1-Pin_2)
- net /r8-2 renamed Net-(JP6-2-Pin_2)
- net /r9-2 renamed Net-(JP6-3-Pin_2)
- net /u12-19 renamed /~{HIGH_DATA_OE}
- net /u13-4 renamed /~{IDE_CS0_OUT}
- J1 pad 78: unconnected-(J1-+5V-Pad78) -> /+5V
- J1 pad 80: unconnected-(J1-GND-Pad80) -> /GND
- J1 pad 9: unconnected-(J1-+12V-Pad9) -> /+12V
- JP6-1 pad 1: unconnected-(JP8-1-Pin_1-Pad1) -> /+5V
- JP6-1 pad 3: unconnected-(JP8-1-Pin_3-Pad3) -> /GND
- JP6-2 pad 1: unconnected-(JP8-2-Pin_1-Pad1) -> /+5V
- JP6-2 pad 3: unconnected-(JP8-2-Pin_3-Pad3) -> /GND
- JP6-3 pad 1: unconnected-(JP8-3-Pin_1-Pad1) -> /+5V
- JP6-3 pad 3: unconnected-(JP8-3-Pin_3-Pad3) -> /GND
- JP6-4 pad 1: unconnected-(JP8-4-Pin_1-Pad1) -> /+5V
- JP6-4 pad 3: unconnected-(JP8-4-Pin_3-Pad3) -> /GND
- JP6-5 pad 1: unconnected-(JP8-5-Pin_1-Pad1) -> /+5V
- JP6-5 pad 3: unconnected-(JP8-5-Pin_3-Pad3) -> /GND
- JP6-6 pad 1: unconnected-(JP8-6-Pin_1-Pad1) -> /+5V
- JP6-6 pad 3: unconnected-(JP8-6-Pin_3-Pad3) -> /GND
- JP6-7 pad 1: unconnected-(JP8-7-Pin_1-Pad1) -> /+5V
- JP6-7 pad 3: unconnected-(JP8-7-Pin_3-Pad3) -> /GND
- JP6-8 pad 1: unconnected-(JP8-8-Pin_1-Pad1) -> /+5V
- JP6-8 pad 3: unconnected-(JP8-8-Pin_3-Pad3) -> /GND
- JP7 pad 1: /+5V -> /GND
- JP7 pad 3: /GND -> /+5V
- JP8 pad 2: unconnected-(JP8-Pin_2-Pad2) -> /U8_IRQ
- JP9-2 pad 1: unconnected-(JP9-2-Pin_1-Pad1) -> /jp9-2
- JP9-2 pad 3: unconnected-(JP9-2-Pin_3-Pad3) -> /jp9-3
- JP9-3 pad 1: unconnected-(JP9-3-Pin_1-Pad1) -> /jp9-2
- JP9-3 pad 3: unconnected-(JP9-3-Pin_3-Pad3) -> /jp9-3
- JP9-4 pad 1: unconnected-(JP9-4-Pin_1-Pad1) -> /jp9-2
- JP9-4 pad 3: unconnected-(JP9-4-Pin_3-Pad3) -> /jp9-3
- JP9-5 pad 1: unconnected-(JP9-5-Pin_1-Pad1) -> /jp9-2
- JP9-5 pad 3: unconnected-(JP9-5-Pin_3-Pad3) -> /jp9-3
- R10 pad 1: unconnected-(R10-Pad1) -> /~{LOW_DATA_OE}
- R12 pad 1: unconnected-(R12-Pad1) -> /u11-31
- R13 pad 1: unconnected-(R13-Pad1) -> /u11-32
- R15 pad 1: /u13-5 -> /~{IDE_CS1_OUT}
- R7 pad 2: unconnected-(R7-Pad2) -> /~{UART1_CS}
- R8 pad 1: unconnected-(R8-Pad1) -> /u11-28
- R9 pad 1: unconnected-(R9-Pad1) -> /~{UART2_CS}
- U11 pad 10: unconnected-(U11-Pad10) -> /~{IOW}
- U11 pad 11: unconnected-(U11-Pad11) -> /RESET
- U11 pad 14: unconnected-(U11-Pad14) -> /u11-14
- U11 pad 15: unconnected-(U11-Pad15) -> /u11-15
- U11 pad 16: unconnected-(U11-Pad16) -> /u11-16
- U11 pad 18: unconnected-(U11-Pad18) -> /u11-18
- U11 pad 19: unconnected-(U11-Pad19) -> /~{BUTTON1}
- U11 pad 20: unconnected-(U11-Pad20) -> /~{BUTTON2}
- U11 pad 21: unconnected-(U11-Pad21) -> /u11-21
- U11 pad 27: /u11-27 -> /~{UART1_CS}
- U11 pad 28: unconnected-(U11-Pad28) -> /u11-28
- U11 pad 29: /u11-29 -> /~{UART2_CS}
- U11 pad 3: unconnected-(U11-Pad3) -> /~{DACK2}
- U11 pad 30: /u11-30 -> /~{LOW_DATA_OE}
- U11 pad 31: unconnected-(U11-Pad31) -> /u11-31
- U11 pad 32: unconnected-(U11-Pad32) -> /u11-32
- U11 pad 45: /u11-45 -> /~{IDE_CS1_OUT}
- U11 pad 5: unconnected-(U11-Pad5) -> /D5
- U11 pad 6: unconnected-(U11-Pad6) -> /D4
- U11 pad 7: unconnected-(U11-Pad7) -> /D1
- U11 pad 8: unconnected-(U11-Pad8) -> /D0
- U11 pad 9: unconnected-(U11-Pad9) -> /~{IOR}
- U12 pad 10: unconnected-(U12-GND-Pad10) -> /GND
- U12 pad 20: unconnected-(U12-VCC-Pad20) -> /+5V
- U13 pad 20: unconnected-(U13-VCC-Pad20) -> /+5V
- U13 pad 5: /u13-5 -> /~{IDE_CS1_OUT}
- U13 pad 6: /u13-6 -> /~{IOW}
- U13 pad 7: /u13-7 -> /~{IOR}
- U14 pad 10: unconnected-(U14-GND-Pad10) -> /GND
- U14 pad 19: /u11-30 -> /~{LOW_DATA_OE}
- U14 pad 20: unconnected-(U14-VCC-Pad20) -> /+5V
- U2 pad 1: unconnected-(U2-Pad1) -> /u4-31
- U2 pad 11: unconnected-(U2-Pad11) -> /~{RESET}
- U2 pad 12: unconnected-(U2-Pad12) -> Net-(R6-Pad1)
- U2 pad 13: unconnected-(U2-Pad13) -> /GND
- U2 pad 14: unconnected-(U2E-VCC-Pad14) -> /+5V
- U2 pad 2: unconnected-(U2-Pad2) -> /u4-30
- U2 pad 3: unconnected-(U2-Pad3) -> /jp9-2
- U2 pad 4: unconnected-(U2-Pad4) -> /u5-31
- U2 pad 5: unconnected-(U2-Pad5) -> /u2-5
- U2 pad 6: unconnected-(U2-Pad6) -> /jp9-3
- U2 pad 7: unconnected-(U2E-GND-Pad7) -> /GND
- U2 pad 8: unconnected-(U2-Pad8) -> Net-(R6-Pad1)
- U2 pad 9: unconnected-(U2-Pad9) -> /+5V
- U4 pad 12: unconnected-(U4-CS0-Pad12) -> /+5V
- U4 pad 13: unconnected-(U4-CS1-Pad13) -> /+5V
- U4 pad 14: unconnected-(U4-~{CS2}-Pad14) -> /~{UART1_CS}
- U4 pad 15: unconnected-(U4-~{BAUDOUT}-Pad15) -> /u4-15
- U4 pad 16: unconnected-(U4-XIN-Pad16) -> /u11-21
- U4 pad 18: unconnected-(U4-~{WR}-Pad18) -> /~{IOW}
- U4 pad 19: unconnected-(U4-WR-Pad19) -> /GND
- U4 pad 2: unconnected-(U4-D1-Pad2) -> /D1
- U4 pad 20: unconnected-(U4-VSS-Pad20) -> /GND
- U4 pad 21: unconnected-(U4-~{RD}-Pad21) -> /~{IOR}
- U4 pad 22: unconnected-(U4-RD-Pad22) -> /GND
- U4 pad 25: unconnected-(U4-~{ADS]-Pad25) -> /GND
- U4 pad 26: unconnected-(U4-A2-Pad26) -> /BA2
- U4 pad 27: unconnected-(U4-A1-Pad27) -> /BA1
- U4 pad 28: unconnected-(U4-A0-Pad28) -> /BA0
- U4 pad 3: unconnected-(U4-D2-Pad3) -> /D2
- U4 pad 30: unconnected-(U4-INTR-Pad30) -> /u4-30
- U4 pad 31: unconnected-(U4-~{OUT2}-Pad31) -> /u4-31
- U4 pad 35: unconnected-(U4-MR-Pad35) -> /RESET
- U4 pad 4: unconnected-(U4-D3-Pad4) -> /D3
- U4 pad 40: unconnected-(U4-VDD-Pad40) -> /+5V
- U4 pad 5: unconnected-(U4-D4-Pad5) -> /D4
- U4 pad 6: unconnected-(U4-D5-Pad6) -> /D5
- U4 pad 7: unconnected-(U4-D6-Pad7) -> /D6
- U4 pad 8: unconnected-(U4-D7-Pad8) -> /D7
- U4 pad 9: unconnected-(U4-RCLK-Pad9) -> /u4-15
- U5 pad 12: unconnected-(U5-CS0-Pad12) -> /+5V
- U5 pad 13: unconnected-(U5-CS1-Pad13) -> /+5V
- U5 pad 14: unconnected-(U5-~{CS2}-Pad14) -> /~{UART2_CS}
- U5 pad 15: unconnected-(U5-~{BAUDOUT}-Pad15) -> /u5-15
- U5 pad 16: unconnected-(U5-XIN-Pad16) -> /u11-21
- U5 pad 18: unconnected-(U5-~{WR}-Pad18) -> /~{IOW}
- U5 pad 19: unconnected-(U5-WR-Pad19) -> /GND
- U5 pad 2: unconnected-(U5-D1-Pad2) -> /D1
- U5 pad 20: unconnected-(U5-VSS-Pad20) -> /GND
- U5 pad 21: unconnected-(U5-~{RD}-Pad21) -> /~{IOR}
- U5 pad 22: unconnected-(U5-RD-Pad22) -> /GND
- U5 pad 25: unconnected-(U5-~{ADS]-Pad25) -> /GND
- U5 pad 26: unconnected-(U5-A2-Pad26) -> /BA2
- U5 pad 27: unconnected-(U5-A1-Pad27) -> /BA1
- U5 pad 28: unconnected-(U5-A0-Pad28) -> /BA0
- U5 pad 3: unconnected-(U5-D2-Pad3) -> /D2
- U5 pad 30: unconnected-(U5-INTR-Pad30) -> /u2-5
- U5 pad 31: unconnected-(U5-~{OUT2}-Pad31) -> /u5-31
- U5 pad 35: unconnected-(U5-MR-Pad35) -> /RESET
- U5 pad 4: unconnected-(U5-D3-Pad4) -> /D3
- U5 pad 40: unconnected-(U5-VDD-Pad40) -> /+5V
- U5 pad 5: unconnected-(U5-D4-Pad5) -> /D4
- U5 pad 6: unconnected-(U5-D5-Pad6) -> /D5
- U5 pad 7: unconnected-(U5-D6-Pad7) -> /D6
- U5 pad 8: unconnected-(U5-D7-Pad8) -> /D7
- U5 pad 9: unconnected-(U5-RCLK-Pad9) -> /u5-15
Routing:
- net /+5V: track 0.00 -> 742.0 mm, vias 0 -> 12
- net /GND: track 11.6 -> 693.0 mm, vias 0 -> 13
- net /D1: track 23.8 -> 230.7 mm, vias 1 -> 3
- net /~{IOW}: track 8.96 -> 213.6 mm, vias 1 -> 7
- net /~{BUTTON1}: track 0.00 -> 199.7 mm, vias 0 -> 1
- net /D4: track 36.3 -> 227.0 mm, vias 1 -> 3
- net /~{BUTTON2}: track 0.00 -> 187.2 mm, vias 0 -> 2
- net /~{IOR}: track 34.7 -> 219.5 mm, vias 0 -> 6
- net /D5: track 41.5 -> 225.3 mm, vias 1 -> 3
- net /u11-14: track 0.00 -> 168.2 mm
- net /D2: track 27.9 -> 190.1 mm, vias 1 -> 3
- net /~{RESET}: track 76.0 -> 237.6 mm, vias 2 -> 4
- net /u11-16: track 0.00 -> 159.6 mm, vias 0 -> 1
- net /D3: track 34.1 -> 190.1 mm, vias 1 -> 3
- net /D7: track 51.8 -> 203.5 mm, vias 1 -> 3
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