File: IDE_controller/IDE_controller/IDE_controller.kicad_sch (KiCad schematic)
At the start: 14 parts, among them J1 Bus_ISA_16bit_narrow, J10 Conn_01x02, U12 74LS245, U13 74LS245

Commit message: IDE controller update
Parts:
- added CON2: Conn_02x17_Odd_Even, Connector_PinHeader_2.54mm:PinHeader_2x17_P2.54mm_Vertical, symbol Connector_Generic:Conn_02x17_Odd_Even
- added JP7, JP8-1, JP8-2, JP8-3, JP8-4, JP8-5, JP8-6, JP8-7, JP8-8: Conn_01x03, Connector_PinHeader_2.54mm:PinHeader_1x03_P2.54mm_Vertical, symbol Connector_Generic:Conn_01x03
- added U11: C820101A, _mine:LQFP-48_10x10mm_P0.7mm, symbol _mine_d:C820101A
Connections:
- net j10-2 is gone; now on net IO_READY: J10.2 (Pin_2)
- net u13-3 is gone; now on net BA2: U13.3 (A1)
- net u13-8 is gone; now on net ALE: U13.8 (A6)
- net BA0: now also U11.23
- net BA1: now also U11.25
- net GND: now also J1.1 (GND), U13.10 (GND), U13.19 (CE), CON2.1 (Pin_1), CON2.11 (Pin_11), CON2.13 (Pin_13), CON2.15 (Pin_15), CON2.17 (Pin_17), CON2.19 (Pin_19), CON2.21 (Pin_21), CON2.23 (Pin_23), CON2.25 (Pin_25), CON2.27 (Pin_27), CON2.29 (Pin_29), CON2.3 (Pin_3), CON2.31 (Pin_31), CON2.33 (Pin_33), CON2.5 (Pin_5), CON2.7 (Pin_7), CON2.9 (Pin_9), JP7.3 (Pin_3), U11.2, U11.34
- net HDD_D10: now also U12.13 (B5)
- net HDD_D11: now also U12.14 (B4)
- net HDD_D12: now also U12.15 (B3)
- net HDD_D8: now also U12.11 (B7)
- net HDD_D9: now also U12.12 (B6)
- net OSC: now also U11.33
- net u12-19: now also R14.1, U11.24
- net u13-4: now also U11.47
- net r7-1: now reaches R7.1
- net r7-1: now also JP8-1.2 (Pin_2)
- net r15-2: now reaches R15.2
- net r15-2: now also JP7.2 (Pin_2)
- net r11-1: now reaches R11.1
- net r11-1: now also U11.4
- net r11-2: now reaches R11.2
- net r11-2: now also JP8-5.2 (Pin_2)
- net r10-2: now reaches R10.2
- net r10-2: now also JP8-4.2 (Pin_2)
- net +5V: now reaches U13.1 (A->B)
- net +5V: now also J1.3 (+5V), JP7.1 (Pin_1), U11.13, U11.35
- net r12-2: now reaches R12.2
- net r12-2: now also JP8-6.2 (Pin_2)
- net r9-2: now reaches R9.2
- net r9-2: now also JP8-3.2 (Pin_2)
- net r14-2: now reaches R14.2
- net r14-2: now also JP8-8.2 (Pin_2)
- net r8-2: now reaches R8.2
- net r8-2: now also JP8-2.2 (Pin_2)
- net RESET: now reaches J1.2 (RESET)
- net IRQ2: now reaches J1.4 (IRQ2)
- net IO_READY: now reaches J1.41 (IO_READY)
- net AEN: now reaches J1.42 (AEN)
- net AEN: now also U11.46
- net BA9: now reaches J1.53 (BA09)
- net BA9: now also U11.43
- net BA8: now reaches J1.54 (BA08)
- net BA8: now also U11.42
- net BA7: now reaches J1.55 (BA07)
- net BA7: now also U11.41
- net BA6: now reaches J1.56 (BA06)
- net BA6: now also U11.40
- net BA5: now reaches J1.57 (BA05)
- net BA5: now also U11.39
- net BA4: now reaches J1.58 (BA04)
- net BA4: now also U11.38
- net BA3: now reaches J1.59 (BA03)
- net BA3: now also U11.37
- net DRQ2: now reaches J1.6 (DRQ2)
- net BA2: now reaches J1.60 (BA02)
- net BA2: now also U11.22
- net -12V: now reaches J1.7 (-12V)
- net r13-2: now reaches R13.2
- net r13-2: now also JP8-7.2 (Pin_2)
- new net u11-27: U11.27
- new net u11-29: U11.29
- new net u11-30: U11.30
- new net u11-45: U11.45
- new net ~{DIR}: CON2.18 (Pin_18)
- new net ~{DS0}: CON2.14 (Pin_14)
- new net ~{DS1}: CON2.12 (Pin_12)
- new net ~{DSKCHNG}: CON2.34 (Pin_34)
- new net ~{HEAD}: CON2.32 (Pin_32)
- new net ~{INDEX}: CON2.8 (Pin_8)
- new net ~{MO0}: CON2.10 (Pin_10)
- new net ~{MO1}: CON2.16 (Pin_16)
- new net ~{RDATA}: CON2.30 (Pin_30)
- new net ~{RWC}: CON2.2 (Pin_2)
- new net ~{STEP}: CON2.20 (Pin_20)
- new net ~{TRAK0}: CON2.26 (Pin_26)
- new net ~{WD}: CON2.22 (Pin_22)
- new net ~{WE}: CON2.24 (Pin_24)
- new net ~{WP}: CON2.28 (Pin_28)
- no-connect marks 28 -> 53

Commit message: IDE controller update
Parts:
- added JP8, JP9-2, JP9-3, JP9-4, JP9-5: Conn_01x03, Connector_PinHeader_2.54mm:PinHeader_1x03_P2.54mm_Vertical, symbol Connector_Generic:Conn_01x03
- added U14: 74LS245, Package_DIP:DIP-20_W7.62mm, symbol 74xx:74LS245
- added U2: 74LS125, Package_DIP:DIP-14_W7.62mm, symbol 74xx:74LS125
- added U4, U5: W86C450, Package_DIP:DIP-40_W15.24mm, symbol _mine_d:W86C450
Connections:
- net HDD_D10 is gone; now on net D10: JP5.8 (Pin_8), U12.13 (B5)
- net HDD_D11 is gone; now on net D11: JP5.10 (Pin_10), U12.14 (B4)
- net HDD_D12 is gone; now on net D12: JP5.12 (Pin_12), U12.15 (B3)
- net HDD_D13 is gone; now on net D13: JP5.14 (Pin_14), U12.16 (B2)
- net HDD_D14 is gone; now on net D14: JP5.16 (Pin_16), U12.17 (B1)
- net HDD_D15 is gone; now on net D15: JP5.18 (Pin_18), U12.18 (B0)
- net HDD_D8 is gone; now on net D8: JP5.4 (Pin_4), U12.11 (B7)
- net HDD_D9 is gone; now on net D9: JP5.6 (Pin_6), U12.12 (B6)
- net +5V: now also J1.29 (VCC)
- net D10: no longer J1.93 (D10), U12.7 (A5)
- net D11: no longer J1.94 (D11), U12.6 (A4)
- net D12: no longer J1.95 (D12), U12.5 (A3)
- net D13: no longer J1.96 (D13), U12.4 (A2)
- net D14: no longer J1.97 (D14), U12.3 (A1)
- net D15: no longer J1.98 (D15), U12.2 (A0)
- net D8: no longer J1.91 (D8), U12.9 (A7)
- net D9: no longer J1.92 (D9), U12.8 (A6)
- net GND: now also J1.10 (GND), J1.31 (GND)
- net IRQ2: now also JP9-2.2 (Pin_2)
- net RESET: now also U2.10
- net u11-30: now also U14.19 (CE)
- net ~{IOR}: now also J1.14 (~{IOR}), U14.1 (A->B); no longer JP5.25 (Pin_25), U12.1 (A->B), U13.13 (B5)
- net ~{IOW}: now also J1.13 (~{IOW}); no longer JP5.23 (Pin_23), U13.14 (B4)
- net IRQ7: now reaches J1.21 (IRQ7)
- net IRQ7: now also JP8.3 (Pin_3)
- net IRQ6: now reaches J1.22 (IRQ6)
- net IRQ5: now reaches J1.23 (IRQ5)
- net IRQ5: now also JP8.1 (Pin_1), JP9-5.2 (Pin_2)
- net IRQ4: now reaches J1.24 (IRQ4)
- net IRQ4: now also JP9-4.2 (Pin_2)
- net IRQ3: now reaches J1.25 (IRQ3)
- net IRQ3: now also JP9-3.2 (Pin_2)
- net ~{DACK2}: now reaches J1.26 (~{DACK2})
- net TC: now reaches J1.27 (TC)
- net DB7: now reaches J1.33 (DB7)
- net DB7: now also U14.9 (A7)
- net DB6: now reaches J1.34 (DB6)
- net DB6: now also U14.8 (A6)
- net DB5: now reaches J1.35 (DB5)
- net DB5: now also U14.7 (A5)
- net DB4: now reaches J1.36 (DB4)
- net DB4: now also U14.6 (A4)
- net DB3: now reaches J1.37 (DB3)
- net DB3: now also U14.5 (A3)
- net DB2: now reaches J1.38 (DB2)
- net DB2: now also U14.4 (A2)
- net DB1: now reaches J1.39 (DB1)
- net DB1: now also U14.3 (A1)
- net DB0: now reaches J1.40 (DB0)
- net DB0: now also U14.2 (A0)
- net BALE renamed ALE_IDE
- net HDD_D0 renamed D0
- net D0: now also U14.18 (B0), U4.1 (D0), U5.1 (D0)
- net HDD_D1 renamed D1
- net D1: now also U14.17 (B1)
- net HDD_D2 renamed D2
- net D2: now also U14.16 (B2)
- net HDD_D3 renamed D3
- net D3: now also U14.15 (B3)
- net HDD_D4 renamed D4
- net D4: now also U14.14 (B4)
- net HDD_D5 renamed D5
- net D5: now also U14.13 (B5)
- net HDD_D6 renamed D6
- net D6: now also U14.12 (B6)
- net HDD_D7 renamed D7
- net D7: now also U14.11 (B7)
- new net DB10: J1.93 (D10), U12.7 (A5)
- new net DB11: J1.94 (D11), U12.6 (A4)
- new net DB12: J1.95 (D12), U12.5 (A3)
- new net DB13: J1.96 (D13), U12.4 (A2)
- new net DB14: J1.97 (D14), U12.3 (A1)
- new net DB15: J1.98 (D15), U12.2 (A0)
- new net DB8: J1.91 (D8), U12.9 (A7)
- new net DB9: J1.92 (D9), U12.8 (A6)
- new net ~{IOR_IDE}: JP5.25 (Pin_25), U12.1 (A->B), U13.13 (B5)
- new net ~{IOW_IDE}: JP5.23 (Pin_23), U13.14 (B4)
- no-connect marks 53 -> 54
Other:
- moved on the sheet: J1, J10, JP5, R10, R11, R12, R13, R14, R15, R7, R8, R9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

Commit message: IDE controller update + decoder
Parts:
- added C1, C10, C11, C12, C13, C14, C2, C3, C4, C5, C6, C8: 100n, Capacitor_THT:C_Disc_D4.3mm_W1.9mm_P5.00mm, symbol Device:C_Small
- added C15, C16: 47p, Capacitor_THT:C_Disc_D4.3mm_W1.9mm_P5.00mm, symbol Device:C_Small
- added C17, C19: 10n, Capacitor_THT:C_Disc_D4.3mm_W1.9mm_P5.00mm, symbol Device:C_Small
- added C18: 470p, Capacitor_THT:C_Disc_D4.3mm_W1.9mm_P5.00mm, symbol Device:C_Small
- added D1: D_Small, Diode_THT:D_A-405_P10.16mm_Horizontal, symbol Device:D_Small
- added J2: DA15_Socket, Connector_Dsub:DSUB-15_Socket_Horizontal_P2.77x2.54mm_EdgePinOffset9.40mm, symbol Connector:DA15_Socket
- added JP1: Conn_01x02, Connector_PinHeader_2.54mm:PinHeader_1x02_P2.54mm_Vertical, symbol Connector_Generic:Conn_01x02
- added R1, R19, R6: 2k2, Resistor_THT:R_Axial_DIN0207_L6.3mm_D2.5mm_P10.16mm_Horizontal, symbol Device:R_Small
- added R16, R17, R2, R20, R3, R5: 4k6, Resistor_THT:R_Axial_DIN0207_L6.3mm_D2.5mm_P10.16mm_Horizontal, symbol Device:R_Small
- added R18, R4: 100R, Resistor_THT:R_Axial_DIN0207_L6.3mm_D2.5mm_P10.16mm_Horizontal, symbol Device:R_Small
- added U8: UM82C11, Package_DIP:DIP-40_W15.24mm, symbol _mine_d:UM82C11
- R10: value 4k6 -> 2k2
- renumbered JP8-1 to JP6-1, JP8-2 to JP6-2, JP8-3 to JP6-3, JP8-4 to JP6-4, JP8-5 to JP6-5, JP8-6 to JP6-6, JP8-7 to JP6-7, JP8-8 to JP6-8
Connections:
- net u11-27 is gone; now on net ~{UART1_CS}: U11.27
- net u11-29 is gone; now on net ~{UART2_CS}: U11.29
- net u11-30 is gone; now on net ~{LOW_DATA_OE}: U11.30, U14.19 (CE)
- net u13-5 is gone; now on net ~{IDE_CS1_OUT}: R15.1, U13.5 (A3)
- net u13-6 is gone; now on net ~{IOW}: U13.6 (A4)
- net u13-7 is gone; now on net ~{IOR}: U13.7 (A5)
- net +5V: now also J1.78 (+5V), JP6-1.1 (Pin_1), JP6-2.1 (Pin_1), JP6-3.1 (Pin_1), JP6-4.1 (Pin_1), JP6-5.1 (Pin_1), JP6-6.1 (Pin_1), JP6-7.1 (Pin_1), JP6-8.1 (Pin_1), JP7.3 (Pin_3), U12.20 (VCC), U13.20 (VCC), U14.20 (VCC), U2.14 (VCC), U2.9, U4.12 (CS0), U4.13 (CS1), U4.40 (VDD), U5.12 (CS0), U5.13 (CS1), U5.40 (VDD), C1.2, C10.2, C11.2, C12.2, C13.2, C14.2, C2.2, C3.2, C4.2, C5.2, C8.2, D1.1 (K), J2.1, J2.15 (P15), J2.8, J2.9 (P9), R16.2, R17.2, R2.2, R20.2, R3.2, R5.2, U8.40 (VDD); no longer JP7.1 (Pin_1)
- net BA0: now also U4.28 (A0), U5.28 (A0), U8.38 (A0)
- net BA1: now also U4.27 (A1), U5.27 (A1), U8.39 (A1)
- net BA2: now also U4.26 (A2), U5.26 (A2)
- net D0: now also U11.8, U8.9 (D0)
- net D1: now also U11.7, U4.2 (D1), U5.2 (D1), U8.10 (D1)
- net D2: now also U4.3 (D2), U5.3 (D2), U8.11 (D2)
- net D3: now also U4.4 (D3), U5.4 (D3), U8.12 (D3)
- net D4: now also U11.6, U4.5 (D4), U5.5 (D4), U8.13 (D4)
- net D5: now also U11.5, U4.6 (D5), U5.6 (D5), U8.14 (D5)
- net D6: now also U4.7 (D6), U5.7 (D6), U8.15 (D6)
- net D7: now also U4.8 (D7), U5.8 (D7), U8.16 (D7)
- net GND: now also J1.80 (GND), JP6-1.3 (Pin_3), JP6-2.3 (Pin_3), JP6-3.3 (Pin_3), JP6-4.3 (Pin_3), JP6-5.3 (Pin_3), JP6-6.3 (Pin_3), JP6-7.3 (Pin_3), JP6-8.3 (Pin_3), JP7.1 (Pin_1), U12.10 (GND), U14.10 (GND), U2.13, U2.7 (GND), U4.19 (WR), U4.20 (VSS), U4.22 (RD), U4.25 (~{ADS}), U5.19 (WR), U5.20 (VSS), U5.22 (RD), U5.25 (~{ADS}), C1.1, C10.1, C11.1, C12.1, C13.1, C14.1, C15.2, C16.2, C17.1, C18.1, C19.1, C2.1, C3.1, C4.1, C5.1, C6.1, C8.1, J2.12 (P12), J2.4, J2.5, R6.2, U8.1 (X1), U8.19 (~{POE}), U8.20 (VSS); no longer JP7.3 (Pin_3)
- net RESET: now also U11.11, U4.35 (MR), U5.35 (MR), C18.2, U8.5 (RST)
- net ~{DACK2}: now also U11.3
- net ~{HDD_ACT}: now also JP1.2 (Pin_2)
- net ~{IOR}: now also U11.9, U4.21 (~{RD}), U5.21 (~{RD}), U8.7 (~{IOR})
- net ~{IOW}: now also U11.10, U4.18 (~{WR}), U5.18 (~{WR}), U8.6 (~{IOW})
- net ~{RESET}: now also U2.11
- net at U2.8: now also U2.12, R6.1
- net u11-14: now reaches U11.14
- net u11-14: now also C17.2, R18.2, R19.1
- net u11-15: now reaches U11.15
- net u11-15: now also R18.1
- net u11-16: now reaches U11.16
- net u11-16: now also C19.2, R1.1, R4.2
- net u11-18: now reaches U11.18
- net u11-18: now also R4.1
- net ~{BUTTON1}: now reaches U11.19
- net ~{BUTTON1}: now also C16.1, J2.2, R2.1
- net ~{BUTTON2}: now reaches U11.20
- net ~{BUTTON2}: now also C15.1, J2.7, R5.1
- net u11-21: now reaches U11.21
- net u11-21: now also U4.16 (XIN), U5.16 (XIN)
- net u11-28: now reaches U11.28
- net u11-28: now also R8.1
- net u11-31: now reaches U11.31
- net u11-31: now also R12.1
- net u11-32: now reaches U11.32
- net u11-32: now also R13.1
- net ~{UART1_CS}: now reaches U4.14 (~{CS2})
- net ~{UART1_CS}: now also R7.2
- net u4-15: now reaches U4.15 (~{BAUDOUT})
- net u4-15: now also U4.9 (RCLK)
- net u4-30: now reaches U4.30 (INTR)
- net u4-30: now also U2.2
- net u4-31: now reaches U4.31 (~{OUT2})
- net u4-31: now also U2.1, R17.1
- net ~{LOW_DATA_OE}: now reaches R10.1
- net jp9-2: now reaches JP9-2.1 (Pin_1)
- net jp9-2: now also JP9-3.1 (Pin_1), JP9-4.1 (Pin_1), JP9-5.1 (Pin_1), U2.3
- net jp9-3: now reaches JP9-2.3 (Pin_3)
- net jp9-3: now also JP9-3.3 (Pin_3), JP9-4.3 (Pin_3), JP9-5.3 (Pin_3), U2.6
- net U8_IRQ: now reaches JP8.2 (Pin_2)
- net U8_IRQ: now also U8.17 (IRQ)
- net ~{UART2_CS}: now reaches R9.1
- net ~{UART2_CS}: now also U5.14 (~{CS2})
- net +12V: now reaches J1.9 (+12V)
- net +12V: now also C6.2
- net u5-31: now reaches U2.4
- net u5-31: now also U5.31 (~{OUT2}), R16.1
- net u2-5: now reaches U2.5
- net u2-5: now also U5.30 (INTR)
- net u5-15: now reaches U5.15 (~{BAUDOUT})
- net u5-15: now also U5.9 (RCLK)
- net r10-2: no longer names the net of JP6-4.2 (Pin_2), R10.2
- net r11-1 renamed U8_CS
- net U8_CS: now also U8.18 (~{CS})
- net r11-2: no longer names the net of JP6-5.2 (Pin_2), R11.2
- net r12-2: no longer names the net of JP6-6.2 (Pin_2), R12.2
- net r13-2: no longer names the net of JP6-7.2 (Pin_2), R13.2
- net r14-2: no longer names the net of JP6-8.2 (Pin_2), R14.2
- net r15-2: no longer names the net of JP7.2 (Pin_2), R15.2
- net r7-1: no longer names the net of JP6-1.2 (Pin_2), R7.1
- net r8-2: no longer names the net of JP6-2.2 (Pin_2), R8.2
- net r9-2: no longer names the net of JP6-3.2 (Pin_2), R9.2
- net u11-45 renamed ~{IDE_CS1_OUT}
- net u12-19 renamed ~{HIGH_DATA_OE}
- net u13-4 renamed ~{IDE_CS0_OUT}
- new net: JP1.1 (Pin_1), R20.1
- new net AXES1_X: J2.3, R1.2
- new net AXES1_Y: J2.6, R19.2
- new net P0: U8.37 (P0)
- new net d1-a: D1.2 (A), R3.1
- no-connect marks 54 -> 75
Other:
- note added: "(1F0 - 1F7)"
- note added: "(3F6 - 3F7)"
- note added: "Hard drive enabled JP7 pins 1 & 2 closed Hard drive disabled JP7 pins 2 & 3 closed"
- note added: "Not Populated"
- note added: "Parallel port is set for IRQ7 JP8 pins 2 & 3 closed Parallel port is set for IRQ5 JP8 pins 1 & 2 closed"
- note added: "SERIAL PORT IRQ JUMPERS - JP9 IRQ Jumper 1 1-2-COM1/3 2-3-COM2/4 Jumper 2 1-2-COM1/3 2-3-COM2/4 Jumper 3 1-2-COM1/3 2-3-COM2/4 Jumper 4 1-2-COM1/3 2-3-COM2/4 5 closed open open open 4 open closed open open 3 open open closed open 2 open open open closed"
- note added: "Serial port 1 is set for COM1 JP6/jumper1 pins 1 & 2 closed (0x3F8-0x3FF) Serial port 1 is set for COM3 JP6/jumper1 pins 2 & 3 closed (0x3E8-0x3EF) Serial port 1 enabled JP6/jumper 2 pins 1 & 2 closed Serial port 1 disabled JP6/jumper 2 pins 2 & 3 closed Serial port 2 is set for COM2 JP6/jumper 3 pins 1 & 2 closed (0x2F8-0x2FF) Serial port 2 is set for COM4 JP6/jumper 3 pins 2 & 3 closed (0x2E8-0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"
- moved on the sheet: J10, JP5, JP6-1, JP6-2, JP6-3, JP6-4, JP6-5, JP6-6, JP6-7, JP6-8, JP7, JP8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
