File: IDE_controller/IDE_controller/IDE_controller.kicad_sch (KiCad schematic)
At the start: 66 parts, among them CON2 Conn_02x17_Odd_Even, J1 Bus_ISA_16bit_narrow, J10 Conn_01x02, J2 DA15_Socket, U11 C820101A, U12 74LS245, U13 74LS245, U14 74LS245, U2 74LS125, U4 W86C450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

Commit message: IDE controller update
Parts:
- removed JP9-2, JP9-3, JP9-4, JP9-5: Conn_01x03, Connector_PinHeader_2.54mm:PinHeader_1x03_P2.54mm_Vertical, symbol Connector_Generic:Conn_01x03
- removed R16, R17: 4k6, Resistor_THT:R_Axial_DIN0207_L6.3mm_D2.5mm_P10.16mm_Horizontal, symbol Device:R_Small
- removed unit 1 of U2
- removed unit 2 of U2
- removed U4, U5: W86C450, Package_DIP:DIP-40_W15.24mm, symbol _mine_d:W86C450
- added U1, U7, U9: SN75189, Package_DIP:DIP-14_W7.62mm, symbol _mine_d:SN75189
- added U6, U8: 74HC00, Package_DIP:DIP-14_W7.62mm, symbol _mine_d:SN75188
- J2: value DA15_Socket -> GAMEPORT
- renumbered U8 to U3
Connections:
- net +12V: now also U6.14 (VCC+), U8.14 (VCC+)
- net +5V: now also U1.14 (VCC), U7.14 (VCC), U9.14 (VCC); no longer C8.2
- net -12V: now also C8.2, U6.1 (VCC-), U8.1 (VCC-)
- net GND: now also U1.7 (GND), U6.7 (GND), U7.7 (GND), U8.7 (GND), U9.7 (GND)
- net U8_CS renamed ~{PARALLEL_CS}
- net u11-14: no longer names the net of C17.2, R18.2, R19.1, U11.14
- net u11-15: no longer names the net of R18.1, U11.15
- net u11-16: no longer names the net of C19.2, R1.1, R4.2, U11.16
- net u11-18: no longer names the net of R4.1, U11.18
- net u11-21 renamed UART_CLK
- no-connect marks 75 -> 78
Other:
- added sheet Serial (Serial.kicad_sch)
- note added: "(1.8MHz)"
- note removed: "SERIAL PORT IRQ JUMPERS - JP9 IRQ Jumper 1 1-2-COM1/3 2-3-COM2/4 Jumper 2 1-2-COM1/3 2-3-COM2/4 Jumper 3 1-2-COM1/3 2-3-COM2/4 Jumper 4 1-2-COM1/3 2-3-COM2/4 5 closed open open open 4 open closed open open 3 open open closed open 2 open open open closed"
- moved on the sheet: C1, C10, C11, C12, C13, C14, C15, C16, C17, C18, C19, C2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
